Commit message: feat: add hand models and update mujoco scenes for g1 robot
- Create MJCF scene files for g1 robot with and without hands
- Update URDF to include hand joints and control logic
- Add hand models in URDF format for left and right hands
- Modify test cases to validate new hand integration
- Introduce a new metapackage for mujoco_ros2_control menagerie

File: ai_worker_mujoco_ros2/ai_worker_mujoco_description/urdf/ai_worker.ros2_control.xacro (robot description, xacro)
@@ -14,4 +14,40 @@
       </state_interface>
     </joint>
+  </xacro:macro>
+  <xacro:macro name="velocity_joint" params="joint_name initial_positions">
+    <joint name="${joint_name}">
+      <command_interface name="velocity"/>
+      <state_interface name="position">
+        <param name="initial_value">${initial_positions[joint_name]}</param>
+      </state_interface>
+      <state_interface name="velocity">
+        <param name="initial_value">0.0</param>
+      </state_interface>
+      <state_interface name="effort">
+        <param name="initial_value">0.0</param>
+      </state_interface>
+    </joint>
+  </xacro:macro>
+  <xacro:macro name="finger_joints" params="side initial_positions">
+    <xacro:position_joint joint_name="finger_${side}_joint1" initial_positions="${initial_positions}"/>
+    <xacro:position_joint joint_name="finger_${side}_joint2" initial_positions="${initial_positions}"/>
+    <xacro:position_joint joint_name="finger_${side}_joint3" initial_positions="${initial_positions}"/>
+    <xacro:position_joint joint_name="finger_${side}_joint4" initial_positions="${initial_positions}"/>
+    <xacro:position_joint joint_name="finger_${side}_joint5" initial_positions="${initial_positions}"/>
+    <xacro:position_joint joint_name="finger_${side}_joint6" initial_positions="${initial_positions}"/>
+    <xacro:position_joint joint_name="finger_${side}_joint7" initial_positions="${initial_positions}"/>
+    <xacro:position_joint joint_name="finger_${side}_joint8" initial_positions="${initial_positions}"/>
+    <xacro:position_joint joint_name="finger_${side}_joint9" initial_positions="${initial_positions}"/>
+    <xacro:position_joint joint_name="finger_${side}_joint10" initial_positions="${initial_positions}"/>
+    <xacro:position_joint joint_name="finger_${side}_joint11" initial_positions="${initial_positions}"/>
+    <xacro:position_joint joint_name="finger_${side}_joint12" initial_positions="${initial_positions}"/>
+    <xacro:position_joint joint_name="finger_${side}_joint13" initial_positions="${initial_positions}"/>
+    <xacro:position_joint joint_name="finger_${side}_joint14" initial_positions="${initial_positions}"/>
+    <xacro:position_joint joint_name="finger_${side}_joint15" initial_positions="${initial_positions}"/>
+    <xacro:position_joint joint_name="finger_${side}_joint16" initial_positions="${initial_positions}"/>
+    <xacro:position_joint joint_name="finger_${side}_joint17" initial_positions="${initial_positions}"/>
+    <xacro:position_joint joint_name="finger_${side}_joint18" initial_positions="${initial_positions}"/>
+    <xacro:position_joint joint_name="finger_${side}_joint19" initial_positions="${initial_positions}"/>
+    <xacro:position_joint joint_name="finger_${side}_joint20" initial_positions="${initial_positions}"/>
   </xacro:macro>
   <xacro:macro name="ai_worker_mujoco_ros2_control" params="name initial_positions_file robot_model">
@@ -41,4 +77,20 @@
       <xacro:position_joint joint_name="arm_r_joint6" initial_positions="${initial_positions}"/>
       <xacro:position_joint joint_name="arm_r_joint7" initial_positions="${initial_positions}"/>
+      <xacro:if value="${robot_model == 'ffw_bg2' or robot_model == 'ffw_sg2'}">
+        <xacro:position_joint joint_name="gripper_l_joint1" initial_positions="${initial_positions}"/>
+        <xacro:position_joint joint_name="gripper_r_joint1" initial_positions="${initial_positions}"/>
+      </xacro:if>
+      <xacro:if value="${robot_model == 'ffw_bh5' or robot_model == 'ffw_sh5'}">
+        <xacro:finger_joints side="l" initial_positions="${initial_positions}"/>
+        <xacro:finger_joints side="r" initial_positions="${initial_positions}"/>
+      </xacro:if>
+      <xacro:if value="${robot_model == 'ffw_sg2' or robot_model == 'ffw_sh5'}">
+        <xacro:position_joint joint_name="left_wheel_steer_joint" initial_positions="${initial_positions}"/>
+        <xacro:position_joint joint_name="right_wheel_steer_joint" initial_positions="${initial_positions}"/>
+        <xacro:position_joint joint_name="rear_wheel_steer_joint" initial_positions="${initial_positions}"/>
+        <xacro:velocity_joint joint_name="left_wheel_drive_joint" initial_positions="${initial_positions}"/>
+        <xacro:velocity_joint joint_name="right_wheel_drive_joint" initial_positions="${initial_positions}"/>
+        <xacro:velocity_joint joint_name="rear_wheel_drive_joint" initial_positions="${initial_positions}"/>
+      </xacro:if>
     </ros2_control>
   </xacro:macro>

File: g1_mujoco_ros2/g1_mujoco_description/urdf/g1.ros2_control.xacro (robot description, xacro)
@@ -15,11 +15,22 @@
     </joint>
   </xacro:macro>
-  <xacro:macro name="g1_mujoco_ros2_control" params="name initial_positions_file mujoco_model_file">
+  <xacro:macro name="g1_hand_joints" params="side initial_positions">
+    <xacro:position_joint joint_name="${side}_hand_thumb_0_joint" initial_positions="${initial_positions}"/>
+    <xacro:position_joint joint_name="${side}_hand_thumb_1_joint" initial_positions="${initial_positions}"/>
+    <xacro:position_joint joint_name="${side}_hand_thumb_2_joint" initial_positions="${initial_positions}"/>
+    <xacro:position_joint joint_name="${side}_hand_middle_0_joint" initial_positions="${initial_positions}"/>
+    <xacro:position_joint joint_name="${side}_hand_middle_1_joint" initial_positions="${initial_positions}"/>
+    <xacro:position_joint joint_name="${side}_hand_index_0_joint" initial_positions="${initial_positions}"/>
+    <xacro:position_joint joint_name="${side}_hand_index_1_joint" initial_positions="${initial_positions}"/>
+  </xacro:macro>
+  <xacro:macro name="g1_mujoco_ros2_control" params="name initial_positions_file robot_model mujoco_model_file">
     <xacro:property name="initial_positions" value="${xacro.load_yaml(initial_positions_file)['initial_positions']}"/>
+    <xacro:property
+      name="selected_mujoco_model_file"
+      value="${mujoco_model_file if mujoco_model_file != 'auto' else ('scene_with_hands.xml' if robot_model == 'g1_with_hands' else 'scene.xml')}"/>
     <ros2_control name="${name}" type="system">
       <hardware>
         <plugin>mujoco_ros2_control/MujocoSystemInterface</plugin>
-        <!-- Package-share equivalent: $(find-pkg-share g1_mujoco_description)/mjcf/g1_29dof_fixed.xml -->
-        <param name="mujoco_model">$(find g1_mujoco_description)/mjcf/${mujoco_model_file}</param>
+        <param name="mujoco_model">$(find g1_mujoco_description)/mjcf/${selected_mujoco_model_file}</param>
         <param name="sim_speed_factor">1.0</param>
         <param name="headless">false</param>
@@ -54,4 +65,8 @@
       <xacro:position_joint joint_name="right_wrist_pitch_joint" initial_positions="${initial_positions}"/>
       <xacro:position_joint joint_name="right_wrist_yaw_joint" initial_positions="${initial_positions}"/>
+      <xacro:if value="${robot_model == 'g1_with_hands'}">
+        <xacro:g1_hand_joints side="left" initial_positions="${initial_positions}"/>
+        <xacro:g1_hand_joints side="right" initial_positions="${initial_positions}"/>
+      </xacro:if>
     </ros2_control>
   </xacro:macro>

File: g1_mujoco_ros2/g1_mujoco_description/urdf/g1_mujoco.urdf.xacro (robot description, xacro)
@@ -2,10 +2,14 @@
 <robot xmlns:xacro="http://www.ros.org/wiki/xacro" name="g1_mujoco">
   <xacro:arg name="initial_positions_file" default="$(find g1_mujoco_description)/config/initial_positions.yaml"/>
-  <xacro:arg name="mujoco_model_file" default="g1_29dof_fixed.xml"/>
+  <xacro:arg name="robot_model" default="g1"/>
+  <xacro:arg name="mujoco_model_file" default="auto"/>
   <xacro:include filename="$(find g1_mujoco_description)/urdf/g1_29dof.urdf"/>
+  <xacro:include filename="$(find g1_mujoco_description)/urdf/g1_hands.urdf.xacro"/>
   <xacro:include filename="$(find g1_mujoco_description)/urdf/g1.ros2_control.xacro"/>
+  <xacro:g1_optional_hands robot_model="$(arg robot_model)"/>
   <xacro:g1_mujoco_ros2_control
     name="g1_mujoco"
     initial_positions_file="$(arg initial_positions_file)"
+    robot_model="$(arg robot_model)"
     mujoco_model_file="$(arg mujoco_model_file)"/>
 </robot>
