Commit message: feat(sim): support headless launches
Expose a common headless launch argument for RBY1, G1, and AI Worker simulations and forward it to the MuJoCo hardware interface.

File: ai_worker_mujoco_ros2/ai_worker_mujoco_description/urdf/ai_worker.ros2_control.xacro (robot description, xacro)
@@ -51,5 +51,5 @@
     <xacro:position_joint joint_name="finger_${side}_joint20" initial_positions="${initial_positions}"/>
   </xacro:macro>
-  <xacro:macro name="ai_worker_mujoco_ros2_control" params="name initial_positions_file robot_model">
+  <xacro:macro name="ai_worker_mujoco_ros2_control" params="name initial_positions_file robot_model headless">
     <xacro:property name="initial_positions" value="${xacro.load_yaml(initial_positions_file)['initial_positions']}"/>
     <ros2_control name="${name}" type="system">
@@ -58,5 +58,5 @@
         <param name="mujoco_model">$(find ai_worker_mujoco_description)/mjcf/scene_${robot_model}.xml</param>
         <param name="sim_speed_factor">1.0</param>
-        <param name="headless">false</param>
+        <param name="headless">${'true' if headless else 'false'}</param>
       </hardware>
       <xacro:position_joint joint_name="lift_joint" initial_positions="${initial_positions}"/>

File: ai_worker_mujoco_ros2/ai_worker_mujoco_description/urdf/ai_worker_mujoco.urdf.xacro (robot description, xacro)
@@ -3,4 +3,5 @@
   <xacro:arg name="robot_model" default="ffw_bg2"/>
   <xacro:arg name="initial_positions_file" default="$(find ai_worker_mujoco_description)/config/initial_positions.yaml"/>
+  <xacro:arg name="headless" default="false"/>
   <xacro:property name="robot_model" value="$(arg robot_model)"/>
   <xacro:if value="${robot_model == 'ffw_bg2'}">
@@ -20,4 +21,5 @@
     name="ai_worker_mujoco"
     initial_positions_file="$(arg initial_positions_file)"
-    robot_model="${robot_model}"/>
+    robot_model="${robot_model}"
+    headless="$(arg headless)"/>
 </robot>

File: g1_mujoco_ros2/g1_mujoco_description/urdf/g1.ros2_control.xacro (robot description, xacro)
@@ -32,5 +32,5 @@
     <xacro:position_joint joint_name="${side}_little_1_joint" initial_positions="${initial_positions}"/>
   </xacro:macro>
-  <xacro:macro name="g1_mujoco_ros2_control" params="name initial_positions_file robot_model mujoco_model_file">
+  <xacro:macro name="g1_mujoco_ros2_control" params="name initial_positions_file robot_model mujoco_model_file headless">
     <xacro:property name="initial_positions" value="${xacro.load_yaml(initial_positions_file)['initial_positions']}"/>
     <xacro:property
@@ -42,5 +42,5 @@
         <param name="mujoco_model">$(find g1_mujoco_description)/mjcf/${selected_mujoco_model_file}</param>
         <param name="sim_speed_factor">1.0</param>
-        <param name="headless">false</param>
+        <param name="headless">${'true' if headless else 'false'}</param>
       </hardware>
       <xacro:position_joint joint_name="left_hip_pitch_joint" initial_positions="${initial_positions}"/>

File: g1_mujoco_ros2/g1_mujoco_description/urdf/g1_mujoco.urdf.xacro (robot description, xacro)
@@ -4,4 +4,5 @@
   <xacro:arg name="robot_model" default="g1"/>
   <xacro:arg name="mujoco_model_file" default="auto"/>
+  <xacro:arg name="headless" default="false"/>
   <xacro:include filename="$(find g1_mujoco_description)/urdf/g1_29dof.urdf"/>
   <xacro:include filename="$(find g1_mujoco_description)/urdf/g1_hands.urdf.xacro"/>
@@ -24,4 +25,5 @@
     initial_positions_file="$(arg initial_positions_file)"
     robot_model="$(arg robot_model)"
-    mujoco_model_file="$(arg mujoco_model_file)"/>
+    mujoco_model_file="$(arg mujoco_model_file)"
+    headless="$(arg headless)"/>
 </robot>

File: rby1_mujoco_ros2/rby1_mujoco_description/urdf/rby1.ros2_control.xacro (robot description, xacro)
@@ -42,5 +42,5 @@
   </xacro:macro>
   <xacro:macro name="rby1_mujoco_ros2_control"
-    params="name robot_model robot_version initial_positions_file">
+    params="name robot_model robot_version initial_positions_file headless">
     <xacro:property name="initial_positions"
       value="${xacro.load_yaml(initial_positions_file)['initial_positions']}" />
@@ -61,5 +61,5 @@
         </xacro:if>
         <param name="sim_speed_factor">1.0</param>
-        <param name="headless">false</param>
+        <param name="headless">${'true' if headless else 'false'}</param>
       </hardware>
       <xacro:if value="${base_robot_model == 'a'}">

File: rby1_mujoco_ros2/rby1_mujoco_description/urdf/rby1.urdf.xacro (robot description, xacro)
@@ -5,4 +5,5 @@
   <xacro:arg name="initial_positions_file"
     default="$(find rby1_mujoco_description)/config/initial_positions/rby1$(arg robot_model).yaml" />
+  <xacro:arg name="headless" default="false" />
   <xacro:arg name="hand_base_offset_z" default="0" />
   <xacro:property name="robot_model" value="$(arg robot_model)" />
@@ -30,4 +31,5 @@
     robot_version="$(arg robot_version)"
     initial_positions_file="$(arg initial_positions_file)"
+    headless="$(arg headless)"
   />
 </robot>
