Commit message: refactor(ai_worker): split body and hand descriptions
- publish full, body-only, and per-hand robot descriptions
- isolate body and hand joint-state publishers by control namespace
- verify all four AI Worker model variants expand consistently

File: ai_worker_mujoco_ros2/ai_worker_mujoco_description/urdf/ai_worker_mujoco.urdf.xacro (robot description, xacro)
@@ -4,4 +4,5 @@
   <xacro:arg name="initial_positions_file" default="$(find ai_worker_mujoco_description)/config/initial_positions.yaml"/>
   <xacro:arg name="headless" default="false"/>
+  <xacro:arg name="include_ros2_control" default="true"/>
   <xacro:property name="robot_model" value="$(arg robot_model)"/>
   <xacro:if value="${robot_model == 'ffw_bg2'}">
@@ -17,9 +18,11 @@
     <xacro:include filename="$(find ai_worker_mujoco_description)/urdf/ffw_sh5_rev1_follower/ffw_sh5_follower.urdf.xacro"/>
   </xacro:if>
-  <xacro:include filename="$(find ai_worker_mujoco_description)/urdf/ai_worker.ros2_control.xacro"/>
-  <xacro:ai_worker_mujoco_ros2_control
-    name="ai_worker_mujoco"
-    initial_positions_file="$(arg initial_positions_file)"
-    robot_model="${robot_model}"
-    headless="$(arg headless)"/>
+  <xacro:if value="$(arg include_ros2_control)">
+    <xacro:include filename="$(find ai_worker_mujoco_description)/urdf/ai_worker.ros2_control.xacro"/>
+    <xacro:ai_worker_mujoco_ros2_control
+      name="ai_worker_mujoco"
+      initial_positions_file="$(arg initial_positions_file)"
+      robot_model="${robot_model}"
+      headless="$(arg headless)"/>
+  </xacro:if>
 </robot>

File: ai_worker_mujoco_ros2/ai_worker_mujoco_description/urdf/ffw_bg2_rev4_follower/ffw_bg2_follower.urdf.xacro (robot description, xacro)
@@ -5,4 +5,5 @@
   <xacro:arg name="prefix" default="" />
   <xacro:arg name="model" default="ffw_bg2_rev4_follower" />
+  <xacro:arg name="include_hands" default="true" />
   <xacro:include filename="$(find ai_worker_mujoco_description)/urdf/common/follower/ffw_follower_body.xacro" />
   <xacro:include filename="$(find ai_worker_mujoco_description)/urdf/common/rh_p12_rn_a/rh_p12_rn_a.urdf.xacro" />
@@ -34,7 +35,9 @@
     <origin xyz="0.0055 0 1.4316" rpy="0 0 0" />
   </xacro:ffw_follower_body>
-  <xacro:rh_p12_rn_a parent="$(arg prefix)arm_l_link7" prefix="$(arg prefix)gripper_l_">
-    <origin xyz="0 0 -0.078" rpy="0 3.14159265359 3.14159265359"/>
-  </xacro:rh_p12_rn_a>
+  <xacro:if value="$(arg include_hands)">
+    <xacro:rh_p12_rn_a parent="$(arg prefix)arm_l_link7" prefix="$(arg prefix)gripper_l_">
+      <origin xyz="0 0 -0.078" rpy="0 3.14159265359 3.14159265359"/>
+    </xacro:rh_p12_rn_a>
+  </xacro:if>
   <joint name="$(arg prefix)end_effector_l_joint" type="fixed">
     <parent link="$(arg prefix)arm_l_link7"/>
@@ -53,7 +56,9 @@
     </visual>
   </link>
-  <xacro:rh_p12_rn_a parent="$(arg prefix)arm_r_link7" prefix="$(arg prefix)gripper_r_">
-    <origin xyz="0 0 -0.078" rpy="0 3.14159265359 3.14159265359"/>
-  </xacro:rh_p12_rn_a>
+  <xacro:if value="$(arg include_hands)">
+    <xacro:rh_p12_rn_a parent="$(arg prefix)arm_r_link7" prefix="$(arg prefix)gripper_r_">
+      <origin xyz="0 0 -0.078" rpy="0 3.14159265359 3.14159265359"/>
+    </xacro:rh_p12_rn_a>
+  </xacro:if>
   <joint name="$(arg prefix)end_effector_r_joint" type="fixed">
     <parent link="$(arg prefix)arm_r_link7"/>

File: ai_worker_mujoco_ros2/ai_worker_mujoco_description/urdf/ffw_bh5_rev1_follower/ffw_bh5_follower.urdf.xacro (robot description, xacro)
@@ -5,4 +5,5 @@
   <xacro:arg name="prefix" default="" />
   <xacro:arg name="model" default="ffw_bh5_rev1_follower" />
+  <xacro:arg name="include_hands" default="true" />
   <xacro:include filename="$(find ai_worker_mujoco_description)/urdf/common/follower/ffw_follower_body.xacro" />
   <xacro:include filename="$(find ai_worker_mujoco_description)/urdf/common/hx5_d20/hx5_d20_left.urdf.xacro" />
@@ -36,9 +37,11 @@
     <origin xyz="0.0055 0 1.4316" rpy="0 0 0" />
   </xacro:ffw_follower_body>
-  <xacro:hx5_d20_left parent="$(arg prefix)arm_l_link7" prefix="$(arg prefix)">
-    <origin xyz="0 0 -0.078" rpy="0 3.14159265359 1.5708"/>
-  </xacro:hx5_d20_left>
-  <xacro:hx5_d20_right parent="$(arg prefix)arm_r_link7" prefix="$(arg prefix)">
-    <origin xyz="0 0 -0.078" rpy="0 3.14159265359 -1.5708"/>
-  </xacro:hx5_d20_right>
+  <xacro:if value="$(arg include_hands)">
+    <xacro:hx5_d20_left parent="$(arg prefix)arm_l_link7" prefix="$(arg prefix)">
+      <origin xyz="0 0 -0.078" rpy="0 3.14159265359 1.5708"/>
+    </xacro:hx5_d20_left>
+    <xacro:hx5_d20_right parent="$(arg prefix)arm_r_link7" prefix="$(arg prefix)">
+      <origin xyz="0 0 -0.078" rpy="0 3.14159265359 -1.5708"/>
+    </xacro:hx5_d20_right>
+  </xacro:if>
 </robot>

File: ai_worker_mujoco_ros2/ai_worker_mujoco_description/urdf/ffw_sg2_rev1_follower/ffw_sg2_follower.urdf.xacro (robot description, xacro)
@@ -5,4 +5,5 @@
   <xacro:arg name="prefix" default="" />
   <xacro:arg name="model" default="ffw_sg2_rev1_follower" />
+  <xacro:arg name="include_hands" default="true" />
   <xacro:include filename="$(find ai_worker_mujoco_description)/urdf/common/follower/ffw_follower_body.xacro" />
   <xacro:include filename="$(find ai_worker_mujoco_description)/urdf/common/rh_p12_rn_a/rh_p12_rn_a.urdf.xacro" />
@@ -107,7 +108,9 @@
     <origin xyz="-0.0199 0 1.4316" rpy="0 0 0" />
   </xacro:ffw_follower_body>
-  <xacro:rh_p12_rn_a parent="$(arg prefix)arm_l_link7" prefix="$(arg prefix)gripper_l_">
-    <origin xyz="0 0 -0.078" rpy="0 3.14159265359 3.14159265359"/>
-  </xacro:rh_p12_rn_a>
+  <xacro:if value="$(arg include_hands)">
+    <xacro:rh_p12_rn_a parent="$(arg prefix)arm_l_link7" prefix="$(arg prefix)gripper_l_">
+      <origin xyz="0 0 -0.078" rpy="0 3.14159265359 3.14159265359"/>
+    </xacro:rh_p12_rn_a>
+  </xacro:if>
   <joint name="$(arg prefix)end_effector_l_joint" type="fixed">
     <parent link="$(arg prefix)arm_l_link7"/>
@@ -126,7 +129,9 @@
     </visual>
   </link>
-  <xacro:rh_p12_rn_a parent="$(arg prefix)arm_r_link7" prefix="$(arg prefix)gripper_r_">
-    <origin xyz="0 0 -0.078" rpy="0 3.14159265359 3.14159265359"/>
-  </xacro:rh_p12_rn_a>
+  <xacro:if value="$(arg include_hands)">
+    <xacro:rh_p12_rn_a parent="$(arg prefix)arm_r_link7" prefix="$(arg prefix)gripper_r_">
+      <origin xyz="0 0 -0.078" rpy="0 3.14159265359 3.14159265359"/>
+    </xacro:rh_p12_rn_a>
+  </xacro:if>
   <joint name="$(arg prefix)end_effector_r_joint" type="fixed">
     <parent link="$(arg prefix)arm_r_link7"/>

File: ai_worker_mujoco_ros2/ai_worker_mujoco_description/urdf/ffw_sh5_rev1_follower/ffw_sh5_follower.urdf.xacro (robot description, xacro)
@@ -5,4 +5,5 @@
   <xacro:arg name="prefix" default="" />
   <xacro:arg name="model" default="ffw_sh5_rev1_follower" />
+  <xacro:arg name="include_hands" default="true" />
   <xacro:include filename="$(find ai_worker_mujoco_description)/urdf/common/follower/ffw_follower_body.xacro" />
   <xacro:include filename="$(find ai_worker_mujoco_description)/urdf/common/hx5_d20/hx5_d20_left.urdf.xacro" />
@@ -86,10 +87,12 @@
     <origin xyz="-0.0199 0 1.4316" rpy="0 0 0" />
   </xacro:ffw_follower_body>
-  <xacro:hx5_d20_left parent="$(arg prefix)arm_l_link7" prefix="$(arg prefix)">
-    <origin xyz="0 0 -0.078" rpy="0 3.14159265359 1.5708"/>
-  </xacro:hx5_d20_left>
-  <xacro:hx5_d20_right parent="$(arg prefix)arm_r_link7" prefix="$(arg prefix)">
-    <origin xyz="0 0 -0.078" rpy="0 3.14159265359 -1.5708"/>
-  </xacro:hx5_d20_right>
+  <xacro:if value="$(arg include_hands)">
+    <xacro:hx5_d20_left parent="$(arg prefix)arm_l_link7" prefix="$(arg prefix)">
+      <origin xyz="0 0 -0.078" rpy="0 3.14159265359 1.5708"/>
+    </xacro:hx5_d20_left>
+    <xacro:hx5_d20_right parent="$(arg prefix)arm_r_link7" prefix="$(arg prefix)">
+      <origin xyz="0 0 -0.078" rpy="0 3.14159265359 -1.5708"/>
+    </xacro:hx5_d20_right>
+  </xacro:if>
   <joint name="$(arg prefix)left_wheel_steer_joint" type="revolute">
       <parent link="$(arg prefix)base_link"/>
