Commit message: feat(rby1): add v1.2 wuji hand variant
- add a single rby1a v1.2 URDF with Wuji hand docking geometry
- attach Wuji hand bodies in MJCF and remove the stock end-effector visuals
- align ros2_control joint order with MuJoCo actuator order for a_wuji
- preserve Wuji hand dynamics by overriding inherited damping and armature

File: rby1_mujoco_ros2/rby1_mujoco_description/urdf/rby1.ros2_control.xacro (robot description, xacro)
@@ -64,7 +64,7 @@
       </hardware>
       <xacro:if value="${base_robot_model == 'a'}">
+        <xacro:velocity_joint joint_name="left_wheel" initial_positions="${initial_positions}"
+          include_temperature="${include_temperature}" />
         <xacro:velocity_joint joint_name="right_wheel" initial_positions="${initial_positions}"
-          include_temperature="${include_temperature}" />
-        <xacro:velocity_joint joint_name="left_wheel" initial_positions="${initial_positions}"
           include_temperature="${include_temperature}" />
         <xacro:position_joint joint_name="torso_0" initial_positions="${initial_positions}"
@@ -137,4 +137,8 @@
       <xacro:position_joint joint_name="left_arm_6" initial_positions="${initial_positions}"
         include_temperature="${include_temperature}" />
+      <xacro:position_joint joint_name="head_0" initial_positions="${initial_positions}"
+        include_temperature="${include_temperature}" />
+      <xacro:position_joint joint_name="head_1" initial_positions="${initial_positions}"
+        include_temperature="${include_temperature}" />
       <xacro:if value="${robot_model != 'a_wuji'}">
         <xacro:position_joint joint_name="right_trigger" initial_positions="${initial_positions}"
@@ -185,8 +189,4 @@
         <xacro:position_joint joint_name="left_finger5_joint4" initial_positions="${initial_positions}" />
       </xacro:if>
-      <xacro:position_joint joint_name="head_0" initial_positions="${initial_positions}"
-        include_temperature="${include_temperature}" />
-      <xacro:position_joint joint_name="head_1" initial_positions="${initial_positions}"
-        include_temperature="${include_temperature}" />
     </ros2_control>
   </xacro:macro>

File: rby1_mujoco_ros2/rby1_mujoco_description/urdf/rby1.urdf.xacro (robot description, xacro)
@@ -11,5 +11,8 @@
   <xacro:property name="gripper_z_offset"
     value="${0 if base_robot_model == 'a' and robot_version == 'v1.0' else -0.035}" />
-  <xacro:if value="${base_robot_model == 'a'}">
+  <xacro:if value="${robot_model == 'a_wuji'}">
+    <xacro:include filename="$(find rby1_mujoco_description)/urdf/rby1a_wuji/model_v1.2.urdf" />
+  </xacro:if>
+  <xacro:if value="${base_robot_model == 'a' and robot_model != 'a_wuji'}">
     <xacro:include filename="$(find rby1_mujoco_description)/urdf/rby1a/model_${robot_version}.urdf" />
   </xacro:if>
@@ -39,18 +42,4 @@
     </joint>
   </xacro:if>
-  <xacro:if value="${robot_model == 'a_wuji'}">
-    <xacro:include filename="$(find rby1_mujoco_description)/urdf/wuji_hand/right.urdf" />
-    <xacro:include filename="$(find rby1_mujoco_description)/urdf/wuji_hand/left.urdf" />
-    <joint name="right_wuji_mount_joint" type="fixed">
-      <parent link="ee_right" />
-      <child link="right_palm_link" />
-      <origin xyz="0 0 -0.2" rpy="3.14159 0 0" />
-    </joint>
-    <joint name="left_wuji_mount_joint" type="fixed">
-      <parent link="ee_left" />
-      <child link="left_palm_link" />
-      <origin xyz="0 0 -0.2" rpy="3.14159 0 0" />
-    </joint>
-  </xacro:if>
   <link name="world" />
   <joint name="world_to_base" type="planar">
