Commit message: feat(rby1): support Hand2 models in MuJoCo bringup
Select Beta1 or Beta2 hands for RBY1A and RBY1M while preserving the Hand1 default. Compose bundled geometry, official collision exclusions, zero initial positions, and matching controller joints at launch.

Add four model/controller checks for A/M and Beta1/Beta2 and document the launch argument. Validation: all four tests pass; launch syntax and diff checks pass.

File: rby1_mujoco_ros2/rby1_mujoco_description/urdf/rby1.ros2_control.xacro (robot description, xacro)
@@ -42,5 +42,5 @@
   </xacro:macro>
   <xacro:macro name="rby1_mujoco_ros2_control"
-    params="name robot_model robot_version initial_positions_file headless">
+    params="name robot_model robot_version initial_positions_file headless hand_model:=wuji_hand mujoco_model_file:=''">
     <xacro:property name="initial_positions"
       value="${xacro.load_yaml(initial_positions_file)['initial_positions']}" />
@@ -51,13 +51,18 @@
       <hardware>
         <plugin>mujoco_ros2_control/MujocoSystemInterface</plugin>
-        <xacro:if value="${robot_model == 'a_wuji'}">
-          <param name="mujoco_model">$(find rby1_mujoco_description)/mjcf/rby1a/model_act_${robot_version}_wuji.xml</param>
+        <xacro:if value="${mujoco_model_file != ''}">
+          <param name="mujoco_model">${mujoco_model_file}</param>
         </xacro:if>
-        <xacro:if value="${robot_model == 'm_wuji'}">
-          <param name="mujoco_model">$(find rby1_mujoco_description)/mjcf/rby1m/model_act_${robot_version}_wuji.xml</param>
-        </xacro:if>
-        <xacro:if value="${(base_robot_model == 'a' or base_robot_model == 'm') and robot_model != 'a_wuji' and robot_model != 'm_wuji'}">
-          <param name="mujoco_model">$(find rby1_mujoco_description)/mjcf/rby1${robot_model}/model_act_${robot_version}.xml</param>
-        </xacro:if>
+        <xacro:unless value="${mujoco_model_file != ''}">
+          <xacro:if value="${robot_model == 'a_wuji'}">
+            <param name="mujoco_model">$(find rby1_mujoco_description)/mjcf/rby1a/model_act_${robot_version}_wuji.xml</param>
+          </xacro:if>
+          <xacro:if value="${robot_model == 'm_wuji'}">
+            <param name="mujoco_model">$(find rby1_mujoco_description)/mjcf/rby1m/model_act_${robot_version}_wuji.xml</param>
+          </xacro:if>
+          <xacro:if value="${(base_robot_model == 'a' or base_robot_model == 'm') and robot_model != 'a_wuji' and robot_model != 'm_wuji'}">
+            <param name="mujoco_model">$(find rby1_mujoco_description)/mjcf/rby1${robot_model}/model_act_${robot_version}.xml</param>
+          </xacro:if>
+        </xacro:unless>
         <param name="sim_speed_factor">1.0</param>
         <param name="headless">${'true' if headless else 'false'}</param>
@@ -135,5 +140,5 @@
       <xacro:position_joint joint_name="head_1" initial_positions="${initial_positions}"
         include_temperature="${include_temperature}" />
-      <xacro:if value="${robot_model == 'a_wuji' or robot_model == 'm_wuji'}">
+      <xacro:if value="${(robot_model == 'a_wuji' or robot_model == 'm_wuji') and hand_model == 'wuji_hand'}">
         <xacro:position_joint joint_name="right_finger1_joint1" initial_positions="${initial_positions}" />
         <xacro:position_joint joint_name="right_finger1_joint2" initial_positions="${initial_positions}" />
@@ -177,4 +182,14 @@
         <xacro:position_joint joint_name="left_finger5_joint4" initial_positions="${initial_positions}" />
       </xacro:if>
+      <xacro:if value="${(robot_model == 'a_wuji' or robot_model == 'm_wuji') and hand_model in ['wuji_hand2_beta1', 'wuji_hand2_beta2']}">
+        <!-- Launch supplies the official Hand2 names and zero initial joint positions. -->
+        <xacro:macro name="hand2_joints" params="names">
+          <xacro:if value="${len(names) > 0}">
+            <xacro:position_joint joint_name="${names[0]}" initial_positions="${initial_positions}" />
+            <xacro:hand2_joints names="${names[1:]}" />
+          </xacro:if>
+        </xacro:macro>
+        <xacro:hand2_joints names="${[n for n in initial_positions if n.startswith('l_') or n.startswith('r_')]}" />
+      </xacro:if>
     </ros2_control>
   </xacro:macro>

File: rby1_mujoco_ros2/rby1_mujoco_description/urdf/rby1.urdf.xacro (robot description, xacro)
@@ -5,4 +5,6 @@
   <xacro:arg name="initial_positions_file"
     default="$(find rby1_mujoco_description)/config/initial_positions/rby1$(arg robot_model).yaml" />
+  <xacro:arg name="hand_model" default="wuji_hand" />
+  <xacro:arg name="mujoco_model_file" default="" />
   <xacro:arg name="headless" default="false" />
   <xacro:arg name="hand_base_offset_z" default="0" />
@@ -19,5 +21,6 @@
   </xacro:if>
   <xacro:if value="${robot_model == 'a_wuji' or robot_model == 'm_wuji'}">
-    <xacro:rby1_wuji_hand_mounts robot_model="${robot_model}" robot_version="${robot_version}" />
+    <xacro:rby1_wuji_hand_mounts robot_model="${robot_model}" robot_version="${robot_version}"
+      hand_model="$(arg hand_model)" />
   </xacro:if>
   <xacro:if value="${robot_model != 'a_wuji' and robot_model != 'm_wuji'}">
@@ -32,4 +35,6 @@
     initial_positions_file="$(arg initial_positions_file)"
     headless="$(arg headless)"
+    hand_model="$(arg hand_model)"
+    mujoco_model_file="$(arg mujoco_model_file)"
   />
 </robot>

File: rby1_mujoco_ros2/rby1_mujoco_description/urdf/wuji_hand/rby1_mount.urdf.xacro (robot description, xacro)
@@ -15,9 +15,27 @@
     </joint>
   </xacro:macro>
-  <xacro:macro name="rby1_wuji_hand_mounts" params="robot_model robot_version">
-    <xacro:include
-      filename="$(find rby1_mujoco_description)/urdf/wuji_hand/right_with_docking.urdf.xacro" />
-    <xacro:include
-      filename="$(find rby1_mujoco_description)/urdf/wuji_hand/left_with_docking.urdf.xacro" />
+  <xacro:macro name="rby1_wuji_hand_mounts" params="robot_model robot_version hand_model:=wuji_hand">
+    <xacro:if value="${hand_model == 'wuji_hand'}">
+      <xacro:include
+        filename="$(find rby1_mujoco_description)/urdf/wuji_hand/right_with_docking.urdf.xacro" />
+      <xacro:include
+        filename="$(find rby1_mujoco_description)/urdf/wuji_hand/left_with_docking.urdf.xacro" />
+    </xacro:if>
+    <xacro:if value="${hand_model in ['wuji_hand2_beta1', 'wuji_hand2_beta2']}">
+      <xacro:include filename="$(find rby1_mujoco_description)/urdf/${hand_model}/right_with_mount-ros.urdf" />
+      <xacro:include filename="$(find rby1_mujoco_description)/urdf/${hand_model}/left_with_mount-ros.urdf" />
+      <link name="right_hand_base" />
+      <link name="left_hand_base" />
+      <joint name="right_wuji_mount_joint" type="fixed">
+        <parent link="right_hand_base" />
+        <child link="r_mount" />
+        <origin xyz="0 0 0" rpy="0 0 0" />
+      </joint>
+      <joint name="left_wuji_mount_joint" type="fixed">
+        <parent link="left_hand_base" />
+        <child link="l_mount" />
+        <origin xyz="0 0 0" rpy="0 0 0" />
+      </joint>
+    </xacro:if>
     <joint name="right_hand_base_joint" type="fixed">
       <parent link="ee_right" />
