Commit message: feat(menagerie): add G1 and RBY1 hand variants
Add hand-enabled G1 URDF variants, including Inspire hand support, and
update bringup to publish robot descriptions for controller tooling.

Replace the old RBY1UB simulation assets with an RBY1M Wuji hand variant,
including MJCF, URDF, mount/docking assets, initial positions, and
ros2_control controller configs.

Refresh the root README and package install rules for the updated model
layout.

File: g1_mujoco_ros2/g1_mujoco_description/urdf/g1_hands.urdf.xacro (robot description, xacro)
@@ -28,7 +28,14 @@
     </joint>
   </xacro:macro>
-  <xacro:macro name="g1_inspire_revolute_joint" params="name parent child xyz axis lower upper">
+  <xacro:macro name="g1_inspire_fixed_joint" params="name parent child xyz rpy">
+    <joint name="${name}" type="fixed">
+      <origin xyz="${xyz}" rpy="${rpy}"/>
+      <parent link="${parent}"/>
+      <child link="${child}"/>
+    </joint>
+  </xacro:macro>
+  <xacro:macro name="g1_inspire_revolute_joint" params="name parent child xyz rpy axis lower upper">
     <joint name="${name}" type="revolute">
-      <origin xyz="${xyz}" rpy="0 0 0"/>
+      <origin xyz="${xyz}" rpy="${rpy}"/>
       <parent link="${parent}"/>
       <child link="${child}"/>
@@ -183,13 +190,20 @@
     <link name="l_ih_thumb_proximal_base"/>
     <link name="l_ih_thumb_proximal"/>
+    <link name="l_ih_thumb_intermediate"/>
+    <link name="l_ih_thumb_distal"/>
     <link name="l_ih_index_proximal"/>
+    <link name="l_ih_index_intermediate"/>
     <link name="l_ih_middle_proximal"/>
+    <link name="l_ih_middle_intermediate"/>
     <link name="l_ih_ring_proximal"/>
+    <link name="l_ih_ring_intermediate"/>
     <link name="l_ih_pinky_proximal"/>
-    <xacro:g1_hand_fixed_joint
+    <link name="l_ih_pinky_intermediate"/>
+    <xacro:g1_inspire_fixed_joint
       name="l_ih_hand_base_joint"
       parent="left_wrist_yaw_link"
       child="l_ih_hand_base"
-      xyz="0.05 0 0"/>
+      xyz="0.05 0 0"
+      rpy="0 0 1.5708"/>
     <xacro:g1_inspire_revolute_joint
       name="l_ih_thumb_proximal_yaw"
@@ -197,4 +211,5 @@
       child="l_ih_thumb_proximal_base"
       xyz="-0.01696 -0.0691 0.02045"
+      rpy="1.5708 0 1.5708"
       axis="0 0 1"
       lower="0"
@@ -205,7 +220,20 @@
       child="l_ih_thumb_proximal"
       xyz="0.0099867 0.0098242 -0.0089"
+      rpy="-1.5708 -0.16939 0"
       axis="0 0 -1"
       lower="0"
       upper="0.6"/>
+    <xacro:g1_inspire_fixed_joint
+      name="l_ih_thumb_intermediate_joint"
+      parent="l_ih_thumb_proximal"
+      child="l_ih_thumb_intermediate"
+      xyz="0.04407 -0.034553 -0.0008"
+      rpy="0 0 0"/>
+    <xacro:g1_inspire_fixed_joint
+      name="l_ih_thumb_distal_joint"
+      parent="l_ih_thumb_intermediate"
+      child="l_ih_thumb_distal"
+      xyz="0.020248 -0.010156 -0.0012"
+      rpy="0 0 0"/>
     <xacro:g1_inspire_revolute_joint
       name="l_ih_index_proximal"
@@ -213,7 +241,14 @@
       child="l_ih_index_proximal"
       xyz="0.00028533 -0.13653 0.032268"
-      axis="0 0 -1"
-      lower="0"
-      upper="1.47"/>
+      rpy="-0.034907 0 0"
+      axis="0 0 -1"
+      lower="0"
+      upper="1.47"/>
+    <xacro:g1_inspire_fixed_joint
+      name="l_ih_index_intermediate_joint"
+      parent="l_ih_index_proximal"
+      child="l_ih_index_intermediate"
+      xyz="-0.0026138 -0.032026 -0.001"
+      rpy="0 0 0"/>
     <xacro:g1_inspire_revolute_joint
       name="l_ih_middle_proximal"
@@ -221,7 +256,14 @@
       child="l_ih_middle_proximal"
       xyz="0.00028533 -0.1371 0.01295"
-      axis="0 0 -1"
-      lower="0"
-      upper="1.47"/>
+      rpy="0 0 0"
+      axis="0 0 -1"
+      lower="0"
+      upper="1.47"/>
+    <xacro:g1_inspire_fixed_joint
+      name="l_ih_middle_intermediate_joint"
+      parent="l_ih_middle_proximal"
+      child="l_ih_middle_intermediate"
+      xyz="-0.0024229 -0.032041 -0.001"
+      rpy="0 0 0"/>
     <xacro:g1_inspire_revolute_joint
       name="l_ih_ring_proximal"
@@ -229,7 +271,14 @@
       child="l_ih_ring_proximal"
       xyz="0.00028533 -0.13691 -0.0062872"
-      axis="0 0 -1"
-      lower="0"
-      upper="1.47"/>
+      rpy="0.05236 0 0"
+      axis="0 0 -1"
+      lower="0"
+      upper="1.47"/>
+    <xacro:g1_inspire_fixed_joint
+      name="l_ih_ring_intermediate_joint"
+      parent="l_ih_ring_proximal"
+      child="l_ih_ring_intermediate"
+      xyz="-0.0024229 -0.032041 -0.001"
+      rpy="0 0 0"/>
     <xacro:g1_inspire_revolute_joint
       name="l_ih_pinky_proximal"
@@ -237,7 +286,14 @@
       child="l_ih_pinky_proximal"
       xyz="0.00028533 -0.13571 -0.025488"
-      axis="0 0 -1"
-      lower="0"
-      upper="1.47"/>
+      rpy="0.10472 0 0"
+      axis="0 0 -1"
+      lower="0"
+      upper="1.47"/>
+    <xacro:g1_inspire_fixed_joint
+      name="l_ih_pinky_intermediate_joint"
+      parent="l_ih_pinky_proximal"
+      child="l_ih_pinky_intermediate"
+      xyz="-0.0024229 -0.032041 -0.001"
+      rpy="0 0 0"/>
   </xacro:macro>
   <xacro:macro name="g1_inspire_right_hand_urdf">
@@ -245,13 +301,20 @@
     <link name="r_ih_thumb_proximal_base"/>
     <link name="r_ih_thumb_proximal"/>
+    <link name="r_ih_thumb_intermediate"/>
+    <link name="r_ih_thumb_distal"/>
     <link name="r_ih_index_proximal"/>
+    <link name="r_ih_index_intermediate"/>
     <link name="r_ih_middle_proximal"/>
+    <link name="r_ih_middle_intermediate"/>
     <link name="r_ih_ring_proximal"/>
+    <link name="r_ih_ring_intermediate"/>
     <link name="r_ih_pinky_proximal"/>
-    <xacro:g1_hand_fixed_joint
+    <link name="r_ih_pinky_intermediate"/>
+    <xacro:g1_inspire_fixed_joint
       name="r_ih_hand_base_joint"
       parent="right_wrist_yaw_link"
       child="r_ih_hand_base"
-      xyz="0.05 0 0"/>
+      xyz="0.05 0 0"
+      rpy="3.14159 0 1.5708"/>
     <xacro:g1_inspire_revolute_joint
       name="r_ih_thumb_proximal_yaw"
@@ -259,4 +322,5 @@
       child="r_ih_thumb_proximal_base"
       xyz="-0.01696 -0.0691 -0.02045"
+      rpy="1.5708 0 -1.5708"
       axis="0 0 -1"
       lower="0"
@@ -267,7 +331,20 @@
       child="r_ih_thumb_proximal"
       xyz="0.0099867 -0.0098242 -0.0089"
+      rpy="1.5708 -0.16939 0"
       axis="0 0 1"
       lower="0"
       upper="0.6"/>
+    <xacro:g1_inspire_fixed_joint
+      name="r_ih_thumb_intermediate_joint"
+      parent="r_ih_thumb_proximal"
+      child="r_ih_thumb_intermediate"
+      xyz="0.04407 0.034553 -0.0008"
+      rpy="0 0 0"/>
+    <xacro:g1_inspire_fixed_joint
+      name="r_ih_thumb_distal_joint"
+      parent="r_ih_thumb_intermediate"
+      child="r_ih_thumb_distal"
+      xyz="0.020248 0.010156 -0.0012"
+      rpy="0 0 0"/>
     <xacro:g1_inspire_revolute_joint
       name="r_ih_index_proximal"
@@ -275,7 +352,14 @@
       child="r_ih_index_proximal"
       xyz="0.00028533 -0.13653 -0.032268"
-      axis="0 0 1"
-      lower="0"
-      upper="1.47"/>
+      rpy="-3.1067 0 0"
+      axis="0 0 1"
+      lower="0"
+      upper="1.47"/>
+    <xacro:g1_inspire_fixed_joint
+      name="r_ih_index_intermediate_joint"
+      parent="r_ih_index_proximal"
+      child="r_ih_index_intermediate"
+      xyz="-0.0026138 0.032026 -0.001"
+      rpy="0 0 0"/>
     <xacro:g1_inspire_revolute_joint
       name="r_ih_middle_proximal"
@@ -283,7 +367,14 @@
       child="r_ih_middle_proximal"
       xyz="0.00028533 -0.1371 -0.01295"
-      axis="0 0 1"
-      lower="0"
-      upper="1.47"/>
+      rpy="3.14159 0 0"
+      axis="0 0 1"
+      lower="0"
+      upper="1.47"/>
+    <xacro:g1_inspire_fixed_joint
+      name="r_ih_middle_intermediate_joint"
+      parent="r_ih_middle_proximal"
+      child="r_ih_middle_intermediate"
+      xyz="-0.0024229 0.032041 -0.001"
+      rpy="0 0 0"/>
     <xacro:g1_inspire_revolute_joint
       name="r_ih_ring_proximal"
@@ -291,7 +382,14 @@
       child="r_ih_ring_proximal"
       xyz="0.00028533 -0.13691 0.0062872"
-      axis="0 0 1"
-      lower="0"
-      upper="1.47"/>
+      rpy="3.0892 0 0"
+      axis="0 0 1"
+      lower="0"
+      upper="1.47"/>
+    <xacro:g1_inspire_fixed_joint
+      name="r_ih_ring_intermediate_joint"
+      parent="r_ih_ring_proximal"
+      child="r_ih_ring_intermediate"
+      xyz="-0.0024229 0.032041 -0.001"
+      rpy="0 0 0"/>
     <xacro:g1_inspire_revolute_joint
       name="r_ih_pinky_proximal"
@@ -299,7 +397,14 @@
       child="r_ih_pinky_proximal"
       xyz="0.00028533 -0.13571 0.025488"
-      axis="0 0 1"
-      lower="0"
-      upper="1.47"/>
+      rpy="3.0369 0 0"
+      axis="0 0 1"
+      lower="0"
+      upper="1.47"/>
+    <xacro:g1_inspire_fixed_joint
+      name="r_ih_pinky_intermediate_joint"
+      parent="r_ih_pinky_proximal"
+      child="r_ih_pinky_intermediate"
+      xyz="-0.0024229 0.032041 -0.001"
+      rpy="0 0 0"/>
   </xacro:macro>
   <xacro:macro name="g1_optional_hands" params="robot_model">

File: rby1_mujoco_ros2/rby1_mujoco_description/urdf/rby1.ros2_control.xacro (robot description, xacro)
@@ -47,5 +47,5 @@
     <xacro:property name="include_temperature" value="false" />
     <xacro:property name="base_robot_model"
-      value="${'a' if robot_model == 'a_wuji' else robot_model}" />
+      value="${'a' if robot_model == 'a_wuji' else ('m' if robot_model == 'm_wuji' else robot_model)}" />
     <ros2_control name="${name}" type="system">
       <hardware>
@@ -54,9 +54,9 @@
           <param name="mujoco_model">$(find rby1_mujoco_description)/mjcf/rby1a/model_act_v1.2_wuji.xml</param>
         </xacro:if>
-        <xacro:if value="${(base_robot_model == 'a' or base_robot_model == 'm') and robot_model != 'a_wuji'}">
+        <xacro:if value="${robot_model == 'm_wuji'}">
+          <param name="mujoco_model">$(find rby1_mujoco_description)/mjcf/rby1m/model_act_v1.2_wuji.xml</param>
+        </xacro:if>
+        <xacro:if value="${(base_robot_model == 'a' or base_robot_model == 'm') and robot_model != 'a_wuji' and robot_model != 'm_wuji'}">
           <param name="mujoco_model">$(find rby1_mujoco_description)/mjcf/rby1${robot_model}/model_act_${robot_version}.xml</param>
-        </xacro:if>
-        <xacro:if value="${base_robot_model == 'ub'}">
-          <param name="mujoco_model">$(find rby1_mujoco_description)/mjcf/rby1${robot_model}/model_act.xml</param>
         </xacro:if>
         <param name="sim_speed_factor">1.0</param>
@@ -103,10 +103,4 @@
           include_temperature="${include_temperature}" />
       </xacro:if>
-      <xacro:if value="${base_robot_model == 'ub'}">
-        <xacro:position_joint joint_name="torso_hp" initial_positions="${initial_positions}"
-          include_temperature="${include_temperature}" />
-        <xacro:position_joint joint_name="torso_5" initial_positions="${initial_positions}"
-          include_temperature="${include_temperature}" />
-      </xacro:if>
       <xacro:position_joint joint_name="right_arm_0" initial_positions="${initial_positions}"
         include_temperature="${include_temperature}" />
@@ -141,5 +135,5 @@
       <xacro:position_joint joint_name="head_1" initial_positions="${initial_positions}"
         include_temperature="${include_temperature}" />
-      <xacro:if value="${robot_model != 'a_wuji'}">
+      <xacro:if value="${robot_model != 'a_wuji' and robot_model != 'm_wuji'}">
         <xacro:position_joint joint_name="right_trigger" initial_positions="${initial_positions}"
           include_temperature="${include_temperature}" />
@@ -147,5 +141,5 @@
           include_temperature="${include_temperature}" />
       </xacro:if>
-      <xacro:if value="${robot_model == 'a_wuji'}">
+      <xacro:if value="${robot_model == 'a_wuji' or robot_model == 'm_wuji'}">
         <xacro:position_joint joint_name="right_finger1_joint1" initial_positions="${initial_positions}" />
         <xacro:position_joint joint_name="right_finger1_joint2" initial_positions="${initial_positions}" />

File: rby1_mujoco_ros2/rby1_mujoco_description/urdf/rby1.urdf.xacro (robot description, xacro)
@@ -8,5 +8,5 @@
   <xacro:property name="robot_version" value="$(arg robot_version)" />
   <xacro:property name="base_robot_model"
-    value="${'a' if robot_model == 'a_wuji' else robot_model}" />
+    value="${'a' if robot_model == 'a_wuji' else ('m' if robot_model == 'm_wuji' else robot_model)}" />
   <xacro:property name="gripper_z_offset"
     value="${0 if base_robot_model == 'a' and robot_version == 'v1.0' else -0.035}" />
@@ -14,15 +14,19 @@
     <xacro:include filename="$(find rby1_mujoco_description)/urdf/rby1a_wuji/model_v1.2.urdf" />
   </xacro:if>
+  <xacro:if value="${robot_model == 'm_wuji'}">
+    <xacro:include filename="$(find rby1_mujoco_description)/urdf/rby1m_wuji/model_v1.2.urdf" />
+  </xacro:if>
   <xacro:if value="${base_robot_model == 'a' and robot_model != 'a_wuji'}">
     <xacro:include filename="$(find rby1_mujoco_description)/urdf/rby1a/model_${robot_version}.urdf" />
   </xacro:if>
-  <xacro:if value="${base_robot_model == 'm'}">
+  <xacro:if value="${base_robot_model == 'm' and robot_model != 'm_wuji'}">
     <xacro:include filename="$(find rby1_mujoco_description)/urdf/rby1m/model_${robot_version}.urdf" />
   </xacro:if>
-  <xacro:if value="${base_robot_model == 'ub'}">
-    <xacro:include filename="$(find rby1_mujoco_description)/urdf/rby1ub/model.urdf" />
+  <xacro:if value="${robot_model == 'a_wuji' or robot_model == 'm_wuji'}">
+    <xacro:include filename="$(find rby1_mujoco_description)/urdf/wuji_hand/rby1_mount.urdf.xacro" />
+    <xacro:rby1_wuji_hand_mounts />
   </xacro:if>
   <!-- Virtual gripper joints for unified ros2_control interfaces. -->
-  <xacro:if value="${robot_model != 'a_wuji'}">
+  <xacro:if value="${robot_model != 'a_wuji' and robot_model != 'm_wuji'}">
     <link name="right_gripper_link" />
     <joint name="right_trigger" type="prismatic">

File: rby1_mujoco_ros2/rby1_mujoco_description/urdf/rby1m_wuji/model_v1.2.urdf (robot description, URDF)
Before this commit: robot rby1a_v1.2_wuji, 32 links, 31 joints
Links:
- removed link wheel_l
- removed link wheel_r
- added link wheel_fl_link, mass 2.54417879; visual mesh filename=package://rby1_mujoco_description/meshes/rby1m/MECANUM_WHEE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
- added link wheel_fr_link, mass 2.54410022; visual mesh filename=package://rby1_mujoco_description/meshes/rby1m/MECANUM_WHEE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
- added link wheel_rl_link, mass 2.54417879; visual mesh filename=package://rby1_mujoco_description/meshes/rby1m/MECANUM_WHEE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
- added link wheel_rr_link, mass 2.54410022; visual mesh filename=package://rby1_mujoco_description/meshes/rby1m/MECANUM_WHEE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
- link base: mass 60.08042639 -> 82.93082168; geometry visual mesh filename=package://rby1_mujoco_description/meshes/rby1m/base.dae
- link link_head_0: geometry visual mesh filename=package://rby1_mujoco_description/meshes/rby1m/NECK_0.dae
- link link_head_1: geometry visual mesh filename=package://rby1_mujoco_description/meshes/rby1m/NECK_1.dae
- link link_head_2: geometry visual mesh filename=package://rby1_mujoco_description/meshes/rby1m/NECK_2.dae
- link link_left_arm_0: geometry collision cylinder length=0.0700 radius=0.075; visual mesh filename=package://rby1_mujoco_description/meshes/rby1m/LINK_14.dae
- link link_left_arm_1: geometry collision cylinder length=0.2000 radius=0.050; visual mesh filename=package://rby1_mujoco_description/meshes/rby1m/LINK_15.dae
- link link_left_arm_2: geometry collision cylinder length=0.080000 radius=0.05; visual mesh filename=package://rby1_mujoco_description/meshes/rby1m/LINK_16.dae
- link link_left_arm_3: geometry collision cylinder length=0.1150 radius=0.04; visual mesh filename=package://rby1_mujoco_description/meshes/rby1m/LINK_17.dae
- link link_left_arm_4: geometry collision cylinder length=0.095000 radius=0.035; visual mesh filename=package://rby1_mujoco_description/meshes/rby1m/LINK_18.dae
- link link_left_arm_5: geometry collision cylinder length=0.2213 radius=0.075; visual mesh filename=package://rby1_mujoco_description/meshes/rby1m/LINK_19_v1.1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
- link link_left_arm_6: geometry visual mesh filename=package://rby1_mujoco_description/meshes/rby1m/LINK_20_v1.1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
- link link_right_arm_0: geometry collision cylinder length=0.0700 radius=0.075; visual mesh filename=package://rby1_mujoco_description/meshes/rby1m/LINK_7.dae
- link link_right_arm_1: geometry collision cylinder length=0.2 radius=0.05; visual mesh filename=package://rby1_mujoco_description/meshes/rby1m/LINK_8.dae
- link link_right_arm_2: geometry collision cylinder length=0.080000 radius=0.05; visual mesh filename=package://rby1_mujoco_description/meshes/rby1m/LINK_9.dae
- link link_right_arm_3: geometry collision cylinder length=0.1150 radius=0.04; visual mesh filename=package://rby1_mujoco_description/meshes/rby1m/LINK_10.dae
- link link_right_arm_4: geometry collision cylinder length=0.095 radius=0.035; visual mesh filename=package://rby1_mujoco_description/meshes/rby1m/LINK_11.dae
- link link_right_arm_5: geometry collision cylinder length=0.2213 radius=0.075; visual mesh filename=package://rby1_mujoco_description/meshes/rby1m/LINK_12_v1.1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
- link link_right_arm_6: geometry visual mesh filename=package://rby1_mujoco_description/meshes/rby1m/LINK_13_v1.1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
- link link_torso_0: geometry collision cylinder length=0.230 radius=0.105; visual mesh filename=package://rby1_mujoco_description/meshes/rby1m/LINK_1.dae
- link link_torso_1: geometry collision cylinder length=0.220 radius=0.115; visual mesh filename=package://rby1_mujoco_description/meshes/rby1m/LINK_2.dae
- link link_torso_2: geometry collision cylinder length=0.1600 radius=0.095; visual mesh filename=package://rby1_mujoco_description/meshes/rby1m/LINK_3.dae
- link link_torso_3: geometry visual mesh filename=package://rby1_mujoco_description/meshes/rby1m/LINK_4.dae
- link link_torso_4: geometry collision cylinder length=0.2 radius=0.105; visual mesh filename=package://rby1_mujoco_description/meshes/rby1m/LINK_5.dae
- link link_torso_5: geometry collision cylinder length=0.1350 radius=0.155; visual mesh filename=package://rby1_mujoco_description/meshes/rby1m/LINK_6.dae
Joints:
- removed joint left_wheel
- removed joint right_wheel
- added joint wheel_fl: type continuous, parent base, child wheel_fl_link, origin xyz=0.243 0.245 0.076 rpy=0.0 0.0 0.0, axis 0 1 0, limit effort=100 velocity=100
- added joint wheel_fr: type continuous, parent base, child wheel_fr_link, origin xyz=0.243 -0.245 0.076 rpy=0.0 0.0 0.0, axis 0 1 0, limit effort=100 velocity=100
- added joint wheel_rl: type continuous, parent base, child wheel_rl_link, origin xyz=-0.247 0.245 0.076 rpy=0.0 0.0 0.0, axis 0 1 0, limit effort=100 velocity=100
- added joint wheel_rr: type continuous, parent base, child wheel_rr_link, origin xyz=-0.247 -0.245 0.076 rpy=0.0 0.0 0.0, axis 0 1 0, limit effort=100 velocity=100
- joint torso_0: origin xyz=0.0 0.0 0.2805 rpy=0.0 0.0 0.0 -> xyz=0.0 0.0 0.2965 rpy=0.0 0.0 0.0
