Commit message: refactor: remove mock components and hardware type from configs
- Exclude mock_components from g1_mujoco_ros2 and rby1_mujoco_ros2
- Remove hardware_type argument from URDF and launch files
- Update controller configurations for rby1 models
- Adjust tests to reflect changes in configurations and dependencies
- Ensure ai_worker_mujoco_ros2 is included in humanoid_mujoco_ros2_control

File: g1_mujoco_ros2/g1_mujoco_description/urdf/g1.ros2_control.xacro (robot description, xacro)
@@ -15,18 +15,13 @@
     </joint>
   </xacro:macro>
-  <xacro:macro name="g1_mujoco_ros2_control" params="name hardware_type initial_positions_file mujoco_model_file">
+  <xacro:macro name="g1_mujoco_ros2_control" params="name initial_positions_file mujoco_model_file">
     <xacro:property name="initial_positions" value="${xacro.load_yaml(initial_positions_file)['initial_positions']}"/>
     <ros2_control name="${name}" type="system">
       <hardware>
-        <xacro:if value="${hardware_type == 'mujoco'}">
-          <plugin>mujoco_ros2_control/MujocoSystemInterface</plugin>
-          <!-- Package-share equivalent: $(find-pkg-share g1_mujoco_description)/mjcf/g1_29dof_fixed.xml -->
-          <param name="mujoco_model">$(find g1_mujoco_description)/mjcf/${mujoco_model_file}</param>
-          <param name="sim_speed_factor">1.0</param>
-          <param name="headless">false</param>
-        </xacro:if>
-        <xacro:if value="${hardware_type == 'mock'}">
-          <plugin>mock_components/GenericSystem</plugin>
-        </xacro:if>
+        <plugin>mujoco_ros2_control/MujocoSystemInterface</plugin>
+        <!-- Package-share equivalent: $(find-pkg-share g1_mujoco_description)/mjcf/g1_29dof_fixed.xml -->
+        <param name="mujoco_model">$(find g1_mujoco_description)/mjcf/${mujoco_model_file}</param>
+        <param name="sim_speed_factor">1.0</param>
+        <param name="headless">false</param>
       </hardware>
       <xacro:position_joint joint_name="left_hip_pitch_joint" initial_positions="${initial_positions}"/>

File: g1_mujoco_ros2/g1_mujoco_description/urdf/g1_mujoco.urdf.xacro (robot description, xacro)
@@ -1,5 +1,4 @@
 <?xml version="1.0"?>
 <robot xmlns:xacro="http://www.ros.org/wiki/xacro" name="g1_mujoco">
-  <xacro:arg name="hardware_type" default="mujoco"/>
   <xacro:arg name="initial_positions_file" default="$(find g1_mujoco_description)/config/initial_positions.yaml"/>
   <xacro:arg name="mujoco_model_file" default="g1_29dof_fixed.xml"/>
@@ -8,5 +7,4 @@
   <xacro:g1_mujoco_ros2_control
     name="g1_mujoco"
-    hardware_type="$(arg hardware_type)"
     initial_positions_file="$(arg initial_positions_file)"
     mujoco_model_file="$(arg mujoco_model_file)"/>

File: rby1_mujoco_ros2/rby1_mujoco_description/urdf/rby1.ros2_control.xacro (robot description, xacro)
@@ -42,5 +42,5 @@
   </xacro:macro>
   <xacro:macro name="rby1_mujoco_ros2_control"
-    params="name robot_model robot_version initial_positions_file hardware_type">
+    params="name robot_model robot_version initial_positions_file">
     <xacro:property name="initial_positions"
       value="${xacro.load_yaml(initial_positions_file)['initial_positions']}" />
@@ -48,18 +48,13 @@
     <ros2_control name="${name}" type="system">
       <hardware>
-        <xacro:if value="${hardware_type == 'mujoco'}">
-          <plugin>mujoco_ros2_control/MujocoSystemInterface</plugin>
-          <xacro:if value="${robot_model == 'a' or robot_model == 'm'}">
-            <param name="mujoco_model">$(find rby1_mujoco_description)/mjcf/rby1${robot_model}/model_act_${robot_version}.xml</param>
-          </xacro:if>
-          <xacro:if value="${robot_model == 'ub'}">
-            <param name="mujoco_model">$(find rby1_mujoco_description)/mjcf/rby1${robot_model}/model_act.xml</param>
-          </xacro:if>
-          <param name="sim_speed_factor">1.0</param>
-          <param name="headless">false</param>
+        <plugin>mujoco_ros2_control/MujocoSystemInterface</plugin>
+        <xacro:if value="${robot_model == 'a' or robot_model == 'm'}">
+          <param name="mujoco_model">$(find rby1_mujoco_description)/mjcf/rby1${robot_model}/model_act_${robot_version}.xml</param>
         </xacro:if>
-        <xacro:if value="${hardware_type == 'mock'}">
-          <plugin>mock_components/GenericSystem</plugin>
+        <xacro:if value="${robot_model == 'ub'}">
+          <param name="mujoco_model">$(find rby1_mujoco_description)/mjcf/rby1${robot_model}/model_act.xml</param>
         </xacro:if>
+        <param name="sim_speed_factor">1.0</param>
+        <param name="headless">false</param>
       </hardware>
       <xacro:if value="${robot_model == 'a'}">

File: rby1_mujoco_ros2/rby1_mujoco_description/urdf/rby1.urdf.xacro (robot description, xacro)
@@ -3,5 +3,4 @@
   <xacro:arg name="robot_model" default="a" />
   <xacro:arg name="robot_version" default="v1.2" />
-  <xacro:arg name="hardware_type" default="mujoco" />
   <xacro:arg name="initial_positions_file"
     default="$(find rby1_mujoco_description)/config/initial_positions/rby1$(arg robot_model).yaml" />
@@ -49,5 +48,4 @@
     robot_version="$(arg robot_version)"
     initial_positions_file="$(arg initial_positions_file)"
-    hardware_type="$(arg hardware_type)"
   />
 </robot>
