Commit message: feat(menagerie): add hand-enabled humanoid variants
- add G1 Inspire hand and RBY1A Wuji hand MuJoCo/ros2_control variants
- include hand meshes, MJCF scenes, controller configs, and initial positions
- update launch model selection and unified control interfaces for hand variants
- consolidate G1 documentation into the root README

File: g1_mujoco_ros2/g1_mujoco_description/urdf/g1.ros2_control.xacro (robot description, xacro)
@@ -24,9 +24,17 @@
     <xacro:position_joint joint_name="${side}_hand_index_1_joint" initial_positions="${initial_positions}"/>
   </xacro:macro>
+  <xacro:macro name="g1_inspire_hand_joints" params="prefix initial_positions">
+    <xacro:position_joint joint_name="${prefix}_thumb_proximal_yaw" initial_positions="${initial_positions}"/>
+    <xacro:position_joint joint_name="${prefix}_thumb_proximal_pitch" initial_positions="${initial_positions}"/>
+    <xacro:position_joint joint_name="${prefix}_index_proximal" initial_positions="${initial_positions}"/>
+    <xacro:position_joint joint_name="${prefix}_middle_proximal" initial_positions="${initial_positions}"/>
+    <xacro:position_joint joint_name="${prefix}_ring_proximal" initial_positions="${initial_positions}"/>
+    <xacro:position_joint joint_name="${prefix}_pinky_proximal" initial_positions="${initial_positions}"/>
+  </xacro:macro>
   <xacro:macro name="g1_mujoco_ros2_control" params="name initial_positions_file robot_model mujoco_model_file">
     <xacro:property name="initial_positions" value="${xacro.load_yaml(initial_positions_file)['initial_positions']}"/>
     <xacro:property
       name="selected_mujoco_model_file"
-      value="${mujoco_model_file if mujoco_model_file != 'auto' else ('scene_with_hands_fixed.xml' if robot_model == 'g1_with_hands' else 'scene.xml')}"/>
+      value="${mujoco_model_file if mujoco_model_file != 'auto' else ('scene_with_hands_fixed.xml' if robot_model == 'g1_with_hands' else ('scene_inspire_hand_fixed.xml' if robot_model == 'g1_with_inspire_hands' else 'scene.xml'))}"/>
     <ros2_control name="${name}" type="system">
       <hardware>
@@ -69,4 +77,8 @@
         <xacro:g1_hand_joints side="right" initial_positions="${initial_positions}"/>
       </xacro:if>
+      <xacro:if value="${robot_model == 'g1_with_inspire_hands'}">
+        <xacro:g1_inspire_hand_joints prefix="l_ih" initial_positions="${initial_positions}"/>
+        <xacro:g1_inspire_hand_joints prefix="r_ih" initial_positions="${initial_positions}"/>
+      </xacro:if>
     </ros2_control>
   </xacro:macro>

File: g1_mujoco_ros2/g1_mujoco_description/urdf/g1_hands.urdf.xacro (robot description, xacro)
@@ -28,4 +28,13 @@
     </joint>
   </xacro:macro>
+  <xacro:macro name="g1_inspire_revolute_joint" params="name parent child xyz axis lower upper">
+    <joint name="${name}" type="revolute">
+      <origin xyz="${xyz}" rpy="0 0 0"/>
+      <parent link="${parent}"/>
+      <child link="${child}"/>
+      <axis xyz="${axis}"/>
+      <limit lower="${lower}" upper="${upper}" effort="1.0" velocity="6.0"/>
+    </joint>
+  </xacro:macro>
   <xacro:macro name="g1_left_hand_urdf">
     <xacro:g1_hand_link name="left_hand_palm_link" mesh="left_hand_palm_link.STL"/>
@@ -170,4 +179,128 @@
       upper="1.74533"/>
   </xacro:macro>
+  <xacro:macro name="g1_inspire_left_hand_urdf">
+    <link name="l_ih_hand_base"/>
+    <link name="l_ih_thumb_proximal_base"/>
+    <link name="l_ih_thumb_proximal"/>
+    <link name="l_ih_index_proximal"/>
+    <link name="l_ih_middle_proximal"/>
+    <link name="l_ih_ring_proximal"/>
+    <link name="l_ih_pinky_proximal"/>
+    <xacro:g1_hand_fixed_joint
+      name="l_ih_hand_base_joint"
+      parent="left_wrist_yaw_link"
+      child="l_ih_hand_base"
+      xyz="0.05 0 0"/>
+    <xacro:g1_inspire_revolute_joint
+      name="l_ih_thumb_proximal_yaw"
+      parent="l_ih_hand_base"
+      child="l_ih_thumb_proximal_base"
+      xyz="-0.01696 -0.0691 0.02045"
+      axis="0 0 1"
+      lower="0"
+      upper="1.308"/>
+    <xacro:g1_inspire_revolute_joint
+      name="l_ih_thumb_proximal_pitch"
+      parent="l_ih_thumb_proximal_base"
+      child="l_ih_thumb_proximal"
+      xyz="0.0099867 0.0098242 -0.0089"
+      axis="0 0 -1"
+      lower="0"
+      upper="0.6"/>
+    <xacro:g1_inspire_revolute_joint
+      name="l_ih_index_proximal"
+      parent="l_ih_hand_base"
+      child="l_ih_index_proximal"
+      xyz="0.00028533 -0.13653 0.032268"
+      axis="0 0 -1"
+      lower="0"
+      upper="1.47"/>
+    <xacro:g1_inspire_revolute_joint
+      name="l_ih_middle_proximal"
+      parent="l_ih_hand_base"
+      child="l_ih_middle_proximal"
+      xyz="0.00028533 -0.1371 0.01295"
+      axis="0 0 -1"
+      lower="0"
+      upper="1.47"/>
+    <xacro:g1_inspire_revolute_joint
+      name="l_ih_ring_proximal"
+      parent="l_ih_hand_base"
+      child="l_ih_ring_proximal"
+      xyz="0.00028533 -0.13691 -0.0062872"
+      axis="0 0 -1"
+      lower="0"
+      upper="1.47"/>
+    <xacro:g1_inspire_revolute_joint
+      name="l_ih_pinky_proximal"
+      parent="l_ih_hand_base"
+      child="l_ih_pinky_proximal"
+      xyz="0.00028533 -0.13571 -0.025488"
+      axis="0 0 -1"
+      lower="0"
+      upper="1.47"/>
+  </xacro:macro>
+  <xacro:macro name="g1_inspire_right_hand_urdf">
+    <link name="r_ih_hand_base"/>
+    <link name="r_ih_thumb_proximal_base"/>
+    <link name="r_ih_thumb_proximal"/>
+    <link name="r_ih_index_proximal"/>
+    <link name="r_ih_middle_proximal"/>
+    <link name="r_ih_ring_proximal"/>
+    <link name="r_ih_pinky_proximal"/>
+    <xacro:g1_hand_fixed_joint
+      name="r_ih_hand_base_joint"
+      parent="right_wrist_yaw_link"
+      child="r_ih_hand_base"
+      xyz="0.05 0 0"/>
+    <xacro:g1_inspire_revolute_joint
+      name="r_ih_thumb_proximal_yaw"
+      parent="r_ih_hand_base"
+      child="r_ih_thumb_proximal_base"
+      xyz="-0.01696 -0.0691 -0.02045"
+      axis="0 0 -1"
+      lower="0"
+      upper="1.308"/>
+    <xacro:g1_inspire_revolute_joint
+      name="r_ih_thumb_proximal_pitch"
+      parent="r_ih_thumb_proximal_base"
+      child="r_ih_thumb_proximal"
+      xyz="0.0099867 -0.0098242 -0.0089"
+      axis="0 0 1"
+      lower="0"
+      upper="0.6"/>
+    <xacro:g1_inspire_revolute_joint
+      name="r_ih_index_proximal"
+      parent="r_ih_hand_base"
+      child="r_ih_index_proximal"
+      xyz="0.00028533 -0.13653 -0.032268"
+      axis="0 0 1"
+      lower="0"
+      upper="1.47"/>
+    <xacro:g1_inspire_revolute_joint
+      name="r_ih_middle_proximal"
+      parent="r_ih_hand_base"
+      child="r_ih_middle_proximal"
+      xyz="0.00028533 -0.1371 -0.01295"
+      axis="0 0 1"
+      lower="0"
+      upper="1.47"/>
+    <xacro:g1_inspire_revolute_joint
+      name="r_ih_ring_proximal"
+      parent="r_ih_hand_base"
+      child="r_ih_ring_proximal"
+      xyz="0.00028533 -0.13691 0.0062872"
+      axis="0 0 1"
+      lower="0"
+      upper="1.47"/>
+    <xacro:g1_inspire_revolute_joint
+      name="r_ih_pinky_proximal"
+      parent="r_ih_hand_base"
+      child="r_ih_pinky_proximal"
+      xyz="0.00028533 -0.13571 0.025488"
+      axis="0 0 1"
+      lower="0"
+      upper="1.47"/>
+  </xacro:macro>
   <xacro:macro name="g1_optional_hands" params="robot_model">
     <xacro:if value="${robot_model == 'g1_with_hands'}">
@@ -175,4 +308,8 @@
       <xacro:g1_right_hand_urdf/>
     </xacro:if>
+    <xacro:if value="${robot_model == 'g1_with_inspire_hands'}">
+      <xacro:g1_inspire_left_hand_urdf/>
+      <xacro:g1_inspire_right_hand_urdf/>
+    </xacro:if>
   </xacro:macro>
 </robot>

File: rby1_mujoco_ros2/rby1_mujoco_description/urdf/rby1.ros2_control.xacro (robot description, xacro)
@@ -46,11 +46,16 @@
       value="${xacro.load_yaml(initial_positions_file)['initial_positions']}" />
     <xacro:property name="include_temperature" value="false" />
+    <xacro:property name="base_robot_model"
+      value="${'a' if robot_model == 'a_wuji' else robot_model}" />
     <ros2_control name="${name}" type="system">
       <hardware>
         <plugin>mujoco_ros2_control/MujocoSystemInterface</plugin>
-        <xacro:if value="${robot_model == 'a' or robot_model == 'm'}">
+        <xacro:if value="${robot_model == 'a_wuji'}">
+          <param name="mujoco_model">$(find rby1_mujoco_description)/mjcf/rby1a/model_act_v1.2_wuji.xml</param>
+        </xacro:if>
+        <xacro:if value="${(base_robot_model == 'a' or base_robot_model == 'm') and robot_model != 'a_wuji'}">
           <param name="mujoco_model">$(find rby1_mujoco_description)/mjcf/rby1${robot_model}/model_act_${robot_version}.xml</param>
         </xacro:if>
-        <xacro:if value="${robot_model == 'ub'}">
+        <xacro:if value="${base_robot_model == 'ub'}">
           <param name="mujoco_model">$(find rby1_mujoco_description)/mjcf/rby1${robot_model}/model_act.xml</param>
         </xacro:if>
@@ -58,5 +63,5 @@
         <param name="headless">false</param>
       </hardware>
-      <xacro:if value="${robot_model == 'a'}">
+      <xacro:if value="${base_robot_model == 'a'}">
         <xacro:velocity_joint joint_name="right_wheel" initial_positions="${initial_positions}"
           include_temperature="${include_temperature}" />
@@ -76,5 +81,5 @@
           include_temperature="${include_temperature}" />
       </xacro:if>
-      <xacro:if value="${robot_model == 'm'}">
+      <xacro:if value="${base_robot_model == 'm'}">
         <xacro:velocity_joint joint_name="wheel_fr" initial_positions="${initial_positions}"
           include_temperature="${include_temperature}" />
@@ -98,5 +103,5 @@
           include_temperature="${include_temperature}" />
       </xacro:if>
-      <xacro:if value="${robot_model == 'ub'}">
+      <xacro:if value="${base_robot_model == 'ub'}">
         <xacro:position_joint joint_name="torso_hp" initial_positions="${initial_positions}"
           include_temperature="${include_temperature}" />
@@ -132,8 +137,52 @@
       <xacro:position_joint joint_name="left_arm_6" initial_positions="${initial_positions}"
         include_temperature="${include_temperature}" />
-      <xacro:position_joint joint_name="right_trigger" initial_positions="${initial_positions}"
-        include_temperature="${include_temperature}" />
-      <xacro:position_joint joint_name="left_trigger" initial_positions="${initial_positions}"
-        include_temperature="${include_temperature}" />
+      <xacro:if value="${robot_model != 'a_wuji'}">
+        <xacro:position_joint joint_name="right_trigger" initial_positions="${initial_positions}"
+          include_temperature="${include_temperature}" />
+        <xacro:position_joint joint_name="left_trigger" initial_positions="${initial_positions}"
+          include_temperature="${include_temperature}" />
+      </xacro:if>
+      <xacro:if value="${robot_model == 'a_wuji'}">
+        <xacro:position_joint joint_name="right_finger1_joint1" initial_positions="${initial_positions}" />
+        <xacro:position_joint joint_name="right_finger1_joint2" initial_positions="${initial_positions}" />
+        <xacro:position_joint joint_name="right_finger1_joint3" initial_positions="${initial_positions}" />
+        <xacro:position_joint joint_name="right_finger1_joint4" initial_positions="${initial_positions}" />
+        <xacro:position_joint joint_name="right_finger2_joint1" initial_positions="${initial_positions}" />
+        <xacro:position_joint joint_name="right_finger2_joint2" initial_positions="${initial_positions}" />
+        <xacro:position_joint joint_name="right_finger2_joint3" initial_positions="${initial_positions}" />
+        <xacro:position_joint joint_name="right_finger2_joint4" initial_positions="${initial_positions}" />
+        <xacro:position_joint joint_name="right_finger3_joint1" initial_positions="${initial_positions}" />
+        <xacro:position_joint joint_name="right_finger3_joint2" initial_positions="${initial_positions}" />
+        <xacro:position_joint joint_name="right_finger3_joint3" initial_positions="${initial_positions}" />
+        <xacro:position_joint joint_name="right_finger3_joint4" initial_positions="${initial_positions}" />
+        <xacro:position_joint joint_name="right_finger4_joint1" initial_positions="${initial_positions}" />
+        <xacro:position_joint joint_name="right_finger4_joint2" initial_positions="${initial_positions}" />
+        <xacro:position_joint joint_name="right_finger4_joint3" initial_positions="${initial_positions}" />
+        <xacro:position_joint joint_name="right_finger4_joint4" initial_positions="${initial_positions}" />
+        <xacro:position_joint joint_name="right_finger5_joint1" initial_positions="${initial_positions}" />
+        <xacro:position_joint joint_name="right_finger5_joint2" initial_positions="${initial_positions}" />
+        <xacro:position_joint joint_name="right_finger5_joint3" initial_positions="${initial_positions}" />
+        <xacro:position_joint joint_name="right_finger5_joint4" initial_positions="${initial_positions}" />
+        <xacro:position_joint joint_name="left_finger1_joint1" initial_positions="${initial_positions}" />
+        <xacro:position_joint joint_name="left_finger1_joint2" initial_positions="${initial_positions}" />
+        <xacro:position_joint joint_name="left_finger1_joint3" initial_positions="${initial_positions}" />
+        <xacro:position_joint joint_name="left_finger1_joint4" initial_positions="${initial_positions}" />
+        <xacro:position_joint joint_name="left_finger2_joint1" initial_positions="${initial_positions}" />
+        <xacro:position_joint joint_name="left_finger2_joint2" initial_positions="${initial_positions}" />
+        <xacro:position_joint joint_name="left_finger2_joint3" initial_positions="${initial_positions}" />
+        <xacro:position_joint joint_name="left_finger2_joint4" initial_positions="${initial_positions}" />
+        <xacro:position_joint joint_name="left_finger3_joint1" initial_positions="${initial_positions}" />
+        <xacro:position_joint joint_name="left_finger3_joint2" initial_positions="${initial_positions}" />
+        <xacro:position_joint joint_name="left_finger3_joint3" initial_positions="${initial_positions}" />
+        <xacro:position_joint joint_name="left_finger3_joint4" initial_positions="${initial_positions}" />
+        <xacro:position_joint joint_name="left_finger4_joint1" initial_positions="${initial_positions}" />
+        <xacro:position_joint joint_name="left_finger4_joint2" initial_positions="${initial_positions}" />
+        <xacro:position_joint joint_name="left_finger4_joint3" initial_positions="${initial_positions}" />
+        <xacro:position_joint joint_name="left_finger4_joint4" initial_positions="${initial_positions}" />
+        <xacro:position_joint joint_name="left_finger5_joint1" initial_positions="${initial_positions}" />
+        <xacro:position_joint joint_name="left_finger5_joint2" initial_positions="${initial_positions}" />
+        <xacro:position_joint joint_name="left_finger5_joint3" initial_positions="${initial_positions}" />
+        <xacro:position_joint joint_name="left_finger5_joint4" initial_positions="${initial_positions}" />
+      </xacro:if>
       <xacro:position_joint joint_name="head_0" initial_positions="${initial_positions}"
         include_temperature="${include_temperature}" />

File: rby1_mujoco_ros2/rby1_mujoco_description/urdf/rby1.urdf.xacro (robot description, xacro)
@@ -7,32 +7,50 @@
   <xacro:property name="robot_model" value="$(arg robot_model)" />
   <xacro:property name="robot_version" value="$(arg robot_version)" />
+  <xacro:property name="base_robot_model"
+    value="${'a' if robot_model == 'a_wuji' else robot_model}" />
   <xacro:property name="gripper_z_offset"
-    value="${0 if robot_model == 'a' and robot_version == 'v1.0' else -0.035}" />
-  <xacro:if value="${robot_model == 'a'}">
+    value="${0 if base_robot_model == 'a' and robot_version == 'v1.0' else -0.035}" />
+  <xacro:if value="${base_robot_model == 'a'}">
     <xacro:include filename="$(find rby1_mujoco_description)/urdf/rby1a/model_${robot_version}.urdf" />
   </xacro:if>
-  <xacro:if value="${robot_model == 'm'}">
+  <xacro:if value="${base_robot_model == 'm'}">
     <xacro:include filename="$(find rby1_mujoco_description)/urdf/rby1m/model_${robot_version}.urdf" />
   </xacro:if>
-  <xacro:if value="${robot_model == 'ub'}">
+  <xacro:if value="${base_robot_model == 'ub'}">
     <xacro:include filename="$(find rby1_mujoco_description)/urdf/rby1ub/model.urdf" />
   </xacro:if>
   <!-- Virtual gripper joints for unified ros2_control interfaces. -->
-  <link name="right_gripper_link" />
-  <joint name="right_trigger" type="prismatic">
-    <parent link="ee_right" />
-    <child link="right_gripper_link" />
-    <origin xyz="0 0 ${gripper_z_offset}" rpy="0 0 0" />
-    <axis xyz="0 0 1" />
-    <limit lower="0" upper="1" effort="1" velocity="10" />
-  </joint>
-  <link name="left_gripper_link" />
-  <joint name="left_trigger" type="prismatic">
-    <parent link="ee_left" />
-    <child link="left_gripper_link" />
-    <origin xyz="0 0 ${gripper_z_offset}" rpy="0 0 0" />
-    <axis xyz="0 0 1" />
-    <limit lower="0" upper="1" effort="1" velocity="10" />
-  </joint>
+  <xacro:if value="${robot_model != 'a_wuji'}">
+    <link name="right_gripper_link" />
+    <joint name="right_trigger" type="prismatic">
+      <parent link="ee_right" />
+      <child link="right_gripper_link" />
+      <origin xyz="0 0 ${gripper_z_offset}" rpy="0 0 0" />
+      <axis xyz="0 0 1" />
+      <limit lower="0" upper="1" effort="1" velocity="10" />
+    </joint>
+    <link name="left_gripper_link" />
+    <joint name="left_trigger" type="prismatic">
+      <parent link="ee_left" />
+      <child link="left_gripper_link" />
+      <origin xyz="0 0 ${gripper_z_offset}" rpy="0 0 0" />
+      <axis xyz="0 0 1" />
+      <limit lower="0" upper="1" effort="1" velocity="10" />
+    </joint>
+  </xacro:if>
+  <xacro:if value="${robot_model == 'a_wuji'}">
+    <xacro:include filename="$(find rby1_mujoco_description)/urdf/wuji_hand/right.urdf" />
+    <xacro:include filename="$(find rby1_mujoco_description)/urdf/wuji_hand/left.urdf" />
+    <joint name="right_wuji_mount_joint" type="fixed">
+      <parent link="ee_right" />
+      <child link="right_palm_link" />
+      <origin xyz="0 0 -0.2" rpy="3.14159 0 0" />
+    </joint>
+    <joint name="left_wuji_mount_joint" type="fixed">
+      <parent link="ee_left" />
+      <child link="left_palm_link" />
+      <origin xyz="0 0 -0.2" rpy="3.14159 0 0" />
+    </joint>
+  </xacro:if>
   <link name="world" />
   <joint name="world_to_base" type="planar">
