Commit message: feat(menagerie): add RH56F1 inspire hand simulation support
- replace G1 inspire hand URDF and MJCF assets with RH56F1 hand models
- expose six active hand joints per side and keep mimic joints passive
- publish split body and hand robot descriptions for G1 and RBY1 variants

File: g1_mujoco_ros2/g1_mujoco_description/urdf/g1.ros2_control.xacro (robot description, xacro)
@@ -24,11 +24,11 @@
     <xacro:position_joint joint_name="${side}_hand_index_1_joint" initial_positions="${initial_positions}"/>
   </xacro:macro>
-  <xacro:macro name="g1_inspire_hand_joints" params="prefix initial_positions">
-    <xacro:position_joint joint_name="${prefix}_thumb_proximal_yaw" initial_positions="${initial_positions}"/>
-    <xacro:position_joint joint_name="${prefix}_thumb_proximal_pitch" initial_positions="${initial_positions}"/>
-    <xacro:position_joint joint_name="${prefix}_index_proximal" initial_positions="${initial_positions}"/>
-    <xacro:position_joint joint_name="${prefix}_middle_proximal" initial_positions="${initial_positions}"/>
-    <xacro:position_joint joint_name="${prefix}_ring_proximal" initial_positions="${initial_positions}"/>
-    <xacro:position_joint joint_name="${prefix}_pinky_proximal" initial_positions="${initial_positions}"/>
+  <xacro:macro name="g1_inspire_hand_joints" params="side initial_positions">
+    <xacro:position_joint joint_name="${side}_thumb_1_joint" initial_positions="${initial_positions}"/>
+    <xacro:position_joint joint_name="${side}_thumb_2_joint" initial_positions="${initial_positions}"/>
+    <xacro:position_joint joint_name="${side}_index_1_joint" initial_positions="${initial_positions}"/>
+    <xacro:position_joint joint_name="${side}_middle_1_joint" initial_positions="${initial_positions}"/>
+    <xacro:position_joint joint_name="${side}_ring_1_joint" initial_positions="${initial_positions}"/>
+    <xacro:position_joint joint_name="${side}_little_1_joint" initial_positions="${initial_positions}"/>
   </xacro:macro>
   <xacro:macro name="g1_mujoco_ros2_control" params="name initial_positions_file robot_model mujoco_model_file">
@@ -78,6 +78,6 @@
       </xacro:if>
       <xacro:if value="${robot_model == 'g1_with_inspire_hands'}">
-        <xacro:g1_inspire_hand_joints prefix="l_ih" initial_positions="${initial_positions}"/>
-        <xacro:g1_inspire_hand_joints prefix="r_ih" initial_positions="${initial_positions}"/>
+        <xacro:g1_inspire_hand_joints side="left" initial_positions="${initial_positions}"/>
+        <xacro:g1_inspire_hand_joints side="right" initial_positions="${initial_positions}"/>
       </xacro:if>
     </ros2_control>

File: g1_mujoco_ros2/g1_mujoco_description/urdf/g1_hands.urdf.xacro (robot description, xacro)
@@ -1,4 +1,5 @@
 <?xml version="1.0"?>
 <robot xmlns:xacro="http://www.ros.org/wiki/xacro">
+  <xacro:include filename="$(find g1_mujoco_description)/urdf/inspire_hand/rh56f1_hand.urdf.xacro"/>
   <xacro:macro name="g1_hand_link" params="name mesh">
     <link name="${name}">
@@ -26,20 +27,4 @@
       <axis xyz="${axis}"/>
       <limit lower="${lower}" upper="${upper}" effort="2.45" velocity="6.0"/>
-    </joint>
-  </xacro:macro>
-  <xacro:macro name="g1_inspire_fixed_joint" params="name parent child xyz rpy">
-    <joint name="${name}" type="fixed">
-      <origin xyz="${xyz}" rpy="${rpy}"/>
-      <parent link="${parent}"/>
-      <child link="${child}"/>
-    </joint>
-  </xacro:macro>
-  <xacro:macro name="g1_inspire_revolute_joint" params="name parent child xyz rpy axis lower upper">
-    <joint name="${name}" type="revolute">
-      <origin xyz="${xyz}" rpy="${rpy}"/>
-      <parent link="${parent}"/>
-      <child link="${child}"/>
-      <axis xyz="${axis}"/>
-      <limit lower="${lower}" upper="${upper}" effort="1.0" velocity="6.0"/>
     </joint>
   </xacro:macro>
@@ -187,224 +172,14 @@
   </xacro:macro>
   <xacro:macro name="g1_inspire_left_hand_urdf">
-    <link name="l_ih_hand_base"/>
-    <link name="l_ih_thumb_proximal_base"/>
-    <link name="l_ih_thumb_proximal"/>
-    <link name="l_ih_thumb_intermediate"/>
-    <link name="l_ih_thumb_distal"/>
-    <link name="l_ih_index_proximal"/>
-    <link name="l_ih_index_intermediate"/>
-    <link name="l_ih_middle_proximal"/>
-    <link name="l_ih_middle_intermediate"/>
-    <link name="l_ih_ring_proximal"/>
-    <link name="l_ih_ring_intermediate"/>
-    <link name="l_ih_pinky_proximal"/>
-    <link name="l_ih_pinky_intermediate"/>
-    <xacro:g1_inspire_fixed_joint
-      name="l_ih_hand_base_joint"
+    <xacro:rh56f1_left_hand
       parent="left_wrist_yaw_link"
-      child="l_ih_hand_base"
-      xyz="0.05 0 0"
-      rpy="0 0 1.5708"/>
-    <xacro:g1_inspire_revolute_joint
-      name="l_ih_thumb_proximal_yaw"
-      parent="l_ih_hand_base"
-      child="l_ih_thumb_proximal_base"
-      xyz="-0.01696 -0.0691 0.02045"
-      rpy="1.5708 0 1.5708"
-      axis="0 0 1"
-      lower="0"
-      upper="1.308"/>
-    <xacro:g1_inspire_revolute_joint
-      name="l_ih_thumb_proximal_pitch"
-      parent="l_ih_thumb_proximal_base"
-      child="l_ih_thumb_proximal"
-      xyz="0.0099867 0.0098242 -0.0089"
-      rpy="-1.5708 -0.16939 0"
-      axis="0 0 -1"
-      lower="0"
-      upper="0.6"/>
-    <xacro:g1_inspire_fixed_joint
-      name="l_ih_thumb_intermediate_joint"
-      parent="l_ih_thumb_proximal"
-      child="l_ih_thumb_intermediate"
-      xyz="0.04407 -0.034553 -0.0008"
-      rpy="0 0 0"/>
-    <xacro:g1_inspire_fixed_joint
-      name="l_ih_thumb_distal_joint"
-      parent="l_ih_thumb_intermediate"
-      child="l_ih_thumb_distal"
-      xyz="0.020248 -0.010156 -0.0012"
-      rpy="0 0 0"/>
-    <xacro:g1_inspire_revolute_joint
-      name="l_ih_index_proximal"
-      parent="l_ih_hand_base"
-      child="l_ih_index_proximal"
-      xyz="0.00028533 -0.13653 0.032268"
-      rpy="-0.034907 0 0"
-      axis="0 0 -1"
-      lower="0"
-      upper="1.47"/>
-    <xacro:g1_inspire_fixed_joint
-      name="l_ih_index_intermediate_joint"
-      parent="l_ih_index_proximal"
-      child="l_ih_index_intermediate"
-      xyz="-0.0026138 -0.032026 -0.001"
-      rpy="0 0 0"/>
-    <xacro:g1_inspire_revolute_joint
-      name="l_ih_middle_proximal"
-      parent="l_ih_hand_base"
-      child="l_ih_middle_proximal"
-      xyz="0.00028533 -0.1371 0.01295"
-      rpy="0 0 0"
-      axis="0 0 -1"
-      lower="0"
-      upper="1.47"/>
-    <xacro:g1_inspire_fixed_joint
-      name="l_ih_middle_intermediate_joint"
-      parent="l_ih_middle_proximal"
-      child="l_ih_middle_intermediate"
-      xyz="-0.0024229 -0.032041 -0.001"
-      rpy="0 0 0"/>
-    <xacro:g1_inspire_revolute_joint
-      name="l_ih_ring_proximal"
-      parent="l_ih_hand_base"
-      child="l_ih_ring_proximal"
-      xyz="0.00028533 -0.13691 -0.0062872"
-      rpy="0.05236 0 0"
-      axis="0 0 -1"
-      lower="0"
-      upper="1.47"/>
-    <xacro:g1_inspire_fixed_joint
-      name="l_ih_ring_intermediate_joint"
-      parent="l_ih_ring_proximal"
-      child="l_ih_ring_intermediate"
-      xyz="-0.0024229 -0.032041 -0.001"
-      rpy="0 0 0"/>
-    <xacro:g1_inspire_revolute_joint
-      name="l_ih_pinky_proximal"
-      parent="l_ih_hand_base"
-      child="l_ih_pinky_proximal"
-      xyz="0.00028533 -0.13571 -0.025488"
-      rpy="0.10472 0 0"
-      axis="0 0 -1"
-      lower="0"
-      upper="1.47"/>
-    <xacro:g1_inspire_fixed_joint
-      name="l_ih_pinky_intermediate_joint"
-      parent="l_ih_pinky_proximal"
-      child="l_ih_pinky_intermediate"
-      xyz="-0.0024229 -0.032041 -0.001"
-      rpy="0 0 0"/>
+      mount_xyz="0.05 0 0"
+      mount_rpy="0 1.5708 0"/>
   </xacro:macro>
   <xacro:macro name="g1_inspire_right_hand_urdf">
-    <link name="r_ih_hand_base"/>
-    <link name="r_ih_thumb_proximal_base"/>
-    <link name="r_ih_thumb_proximal"/>
-    <link name="r_ih_thumb_intermediate"/>
-    <link name="r_ih_thumb_distal"/>
-    <link name="r_ih_index_proximal"/>
-    <link name="r_ih_index_intermediate"/>
-    <link name="r_ih_middle_proximal"/>
-    <link name="r_ih_middle_intermediate"/>
-    <link name="r_ih_ring_proximal"/>
-    <link name="r_ih_ring_intermediate"/>
-    <link name="r_ih_pinky_proximal"/>
-    <link name="r_ih_pinky_intermediate"/>
-    <xacro:g1_inspire_fixed_joint
-      name="r_ih_hand_base_joint"
+    <xacro:rh56f1_right_hand
       parent="right_wrist_yaw_link"
-      child="r_ih_hand_base"
-      xyz="0.05 0 0"
-      rpy="3.14159 0 1.5708"/>
-    <xacro:g1_inspire_revolute_joint
-      name="r_ih_thumb_proximal_yaw"
-      parent="r_ih_hand_base"
-      child="r_ih_thumb_proximal_base"
-      xyz="-0.01696 -0.0691 -0.02045"
-      rpy="1.5708 0 -1.5708"
-      axis="0 0 -1"
-      lower="0"
-      upper="1.308"/>
-    <xacro:g1_inspire_revolute_joint
-      name="r_ih_thumb_proximal_pitch"
-      parent="r_ih_thumb_proximal_base"
-      child="r_ih_thumb_proximal"
-      xyz="0.0099867 -0.0098242 -0.0089"
-      rpy="1.5708 -0.16939 0"
-      axis="0 0 1"
-      lower="0"
-      upper="0.6"/>
-    <xacro:g1_inspire_fixed_joint
-      name="r_ih_thumb_intermediate_joint"
-      parent="r_ih_thumb_proximal"
-      child="r_ih_thumb_intermediate"
-      xyz="0.04407 0.034553 -0.0008"
-      rpy="0 0 0"/>
-    <xacro:g1_inspire_fixed_joint
-      name="r_ih_thumb_distal_joint"
-      parent="r_ih_thumb_intermediate"
-      child="r_ih_thumb_distal"
-      xyz="0.020248 0.010156 -0.0012"
-      rpy="0 0 0"/>
-    <xacro:g1_inspire_revolute_joint
-      name="r_ih_index_proximal"
-      parent="r_ih_hand_base"
-      child="r_ih_index_proximal"
-      xyz="0.00028533 -0.13653 -0.032268"
-      rpy="-3.1067 0 0"
-      axis="0 0 1"
-      lower="0"
-      upper="1.47"/>
-    <xacro:g1_inspire_fixed_joint
-      name="r_ih_index_intermediate_joint"
-      parent="r_ih_index_proximal"
-      child="r_ih_index_intermediate"
-      xyz="-0.0026138 0.032026 -0.001"
-      rpy="0 0 0"/>
-    <xacro:g1_inspire_revolute_joint
-      name="r_ih_middle_proximal"
-      parent="r_ih_hand_base"
-      child="r_ih_middle_proximal"
-      xyz="0.00028533 -0.1371 -0.01295"
-      rpy="3.14159 0 0"
-      axis="0 0 1"
-      lower="0"
-      upper="1.47"/>
-    <xacro:g1_inspire_fixed_joint
-      name="r_ih_middle_intermediate_joint"
-      parent="r_ih_middle_proximal"
-      child="r_ih_middle_intermediate"
-      xyz="-0.0024229 0.032041 -0.001"
-      rpy="0 0 0"/>
-    <xacro:g1_inspire_revolute_joint
-      name="r_ih_ring_proximal"
-      parent="r_ih_hand_base"
-      child="r_ih_ring_proximal"
-      xyz="0.00028533 -0.13691 0.0062872"
-      rpy="3.0892 0 0"
-      axis="0 0 1"
-      lower="0"
-      upper="1.47"/>
-    <xacro:g1_inspire_fixed_joint
-      name="r_ih_ring_intermediate_joint"
-      parent="r_ih_ring_proximal"
-      child="r_ih_ring_intermediate"
-      xyz="-0.0024229 0.032041 -0.001"
-      rpy="0 0 0"/>
-    <xacro:g1_inspire_revolute_joint
-      name="r_ih_pinky_proximal"
-      parent="r_ih_hand_base"
-      child="r_ih_pinky_proximal"
-      xyz="0.00028533 -0.13571 0.025488"
-      rpy="3.0369 0 0"
-      axis="0 0 1"
-      lower="0"
-      upper="1.47"/>
-    <xacro:g1_inspire_fixed_joint
-      name="r_ih_pinky_intermediate_joint"
-      parent="r_ih_pinky_proximal"
-      child="r_ih_pinky_intermediate"
-      xyz="-0.0024229 0.032041 -0.001"
-      rpy="0 0 0"/>
+      mount_xyz="0.05 0 0"
+      mount_rpy="0 1.5708 0"/>
   </xacro:macro>
   <xacro:macro name="g1_optional_hands" params="robot_model">
