Commit message: refactor(menagerie): align hand mounts and prune stale assets
- Align G1 hand_base frames and mount Inspire hands through body-defined attachment frames
- Preserve g1_with_hands via adapter frames while removing unused rubber hand references
- Clean generated AI Worker URDFs and stale Inspire/RBY1 gripper mesh assets
- Update RBY1 Wuji hand integration around split body and hand descriptions

File: g1_mujoco_ros2/g1_mujoco_description/urdf/g1_29dof.urdf (robot description, URDF)
Before this commit: robot g1_29dof, 40 links, 39 joints
Links:
- removed link left_rubber_hand
- removed link right_rubber_hand
Joints:
- removed joint left_hand_palm_joint
- removed joint right_hand_palm_joint

File: g1_mujoco_ros2/g1_mujoco_description/urdf/g1_hand_left.urdf.xacro (robot description, xacro)
@@ -1,5 +1,5 @@
 <?xml version="1.0"?>
 <robot xmlns:xacro="http://www.ros.org/wiki/xacro" name="g1_hand_left">
-  <link name="left_wrist_yaw_link"/>
+  <link name="left_hand_base"/>
   <xacro:include filename="$(find g1_mujoco_description)/urdf/g1_hands.urdf.xacro"/>
   <xacro:g1_left_hand_urdf/>

File: g1_mujoco_ros2/g1_mujoco_description/urdf/g1_hand_right.urdf.xacro (robot description, xacro)
@@ -1,5 +1,5 @@
 <?xml version="1.0"?>
 <robot xmlns:xacro="http://www.ros.org/wiki/xacro" name="g1_hand_right">
-  <link name="right_wrist_yaw_link"/>
+  <link name="right_hand_base"/>
   <xacro:include filename="$(find g1_mujoco_description)/urdf/g1_hands.urdf.xacro"/>
   <xacro:g1_right_hand_urdf/>

File: g1_mujoco_ros2/g1_mujoco_description/urdf/g1_hands.urdf.xacro (robot description, xacro)
@@ -30,4 +30,10 @@
   </xacro:macro>
   <xacro:macro name="g1_left_hand_urdf">
+    <link name="left_g1_hand_mount"/>
+    <joint name="left_g1_hand_mount_joint" type="fixed">
+      <origin xyz="0 0 0.05" rpy="0 1.57079632679 0"/>
+      <parent link="left_hand_base"/>
+      <child link="left_g1_hand_mount"/>
+    </joint>
     <xacro:g1_hand_link name="left_hand_palm_link" mesh="left_hand_palm_link.STL"/>
     <xacro:g1_hand_link name="left_hand_thumb_0_link" mesh="left_hand_thumb_0_link.STL"/>
@@ -40,10 +46,10 @@
     <xacro:g1_hand_fixed_joint
       name="left_hand_palm_mount_joint"
-      parent="left_wrist_yaw_link"
+      parent="left_g1_hand_mount"
       child="left_hand_palm_link"
       xyz="0.0415 0.003 0"/>
     <xacro:g1_hand_revolute_joint
       name="left_hand_thumb_0_joint"
-      parent="left_wrist_yaw_link"
+      parent="left_g1_hand_mount"
       child="left_hand_thumb_0_link"
       xyz="0.067 0.003 0"
@@ -69,5 +75,5 @@
     <xacro:g1_hand_revolute_joint
       name="left_hand_middle_0_joint"
-      parent="left_wrist_yaw_link"
+      parent="left_g1_hand_mount"
       child="left_hand_middle_0_link"
       xyz="0.1192 0.0046 -0.0285"
@@ -85,5 +91,5 @@
     <xacro:g1_hand_revolute_joint
       name="left_hand_index_0_joint"
-      parent="left_wrist_yaw_link"
+      parent="left_g1_hand_mount"
       child="left_hand_index_0_link"
       xyz="0.1192 0.0046 0.0285"
@@ -101,4 +107,10 @@
   </xacro:macro>
   <xacro:macro name="g1_right_hand_urdf">
+    <link name="right_g1_hand_mount"/>
+    <joint name="right_g1_hand_mount_joint" type="fixed">
+      <origin xyz="0 0 0.05" rpy="0 1.57079632679 0"/>
+      <parent link="right_hand_base"/>
+      <child link="right_g1_hand_mount"/>
+    </joint>
     <xacro:g1_hand_link name="right_hand_palm_link" mesh="right_hand_palm_link.STL"/>
     <xacro:g1_hand_link name="right_hand_thumb_0_link" mesh="right_hand_thumb_0_link.STL"/>
@@ -111,10 +123,10 @@
     <xacro:g1_hand_fixed_joint
       name="right_hand_palm_mount_joint"
-      parent="right_wrist_yaw_link"
+      parent="right_g1_hand_mount"
       child="right_hand_palm_link"
       xyz="0.0415 -0.003 0"/>
     <xacro:g1_hand_revolute_joint
       name="right_hand_thumb_0_joint"
-      parent="right_wrist_yaw_link"
+      parent="right_g1_hand_mount"
       child="right_hand_thumb_0_link"
       xyz="0.067 -0.003 0"
@@ -140,5 +152,5 @@
     <xacro:g1_hand_revolute_joint
       name="right_hand_middle_0_joint"
-      parent="right_wrist_yaw_link"
+      parent="right_g1_hand_mount"
       child="right_hand_middle_0_link"
       xyz="0.1192 -0.0046 -0.0285"
@@ -156,5 +168,5 @@
     <xacro:g1_hand_revolute_joint
       name="right_hand_index_0_joint"
-      parent="right_wrist_yaw_link"
+      parent="right_g1_hand_mount"
       child="right_hand_index_0_link"
       xyz="0.1192 -0.0046 0.0285"
@@ -173,13 +185,13 @@
   <xacro:macro name="g1_inspire_left_hand_urdf">
     <xacro:rh56f1_left_hand
-      parent="left_wrist_yaw_link"
-      mount_xyz="0.05 0 0"
-      mount_rpy="0 1.5708 0"/>
+      parent="left_hand_base"
+      mount_xyz="0 0 0"
+      mount_rpy="0 0 0"/>
   </xacro:macro>
   <xacro:macro name="g1_inspire_right_hand_urdf">
     <xacro:rh56f1_right_hand
-      parent="right_wrist_yaw_link"
-      mount_xyz="0.05 0 0"
-      mount_rpy="0 1.5708 0"/>
+      parent="right_hand_base"
+      mount_xyz="0 0 0"
+      mount_rpy="0 0 0"/>
   </xacro:macro>
   <xacro:macro name="g1_optional_hands" params="robot_model">

File: g1_mujoco_ros2/g1_mujoco_description/urdf/g1_inspire_hand_left.urdf.xacro (robot description, xacro)
@@ -1,5 +1,5 @@
 <?xml version="1.0"?>
 <robot xmlns:xacro="http://www.ros.org/wiki/xacro" name="g1_inspire_hand_left">
-  <link name="left_wrist_yaw_link"/>
+  <link name="left_hand_base"/>
   <xacro:include filename="$(find g1_mujoco_description)/urdf/g1_hands.urdf.xacro"/>
   <xacro:g1_inspire_left_hand_urdf/>

File: g1_mujoco_ros2/g1_mujoco_description/urdf/g1_inspire_hand_right.urdf.xacro (robot description, xacro)
@@ -1,5 +1,5 @@
 <?xml version="1.0"?>
 <robot xmlns:xacro="http://www.ros.org/wiki/xacro" name="g1_inspire_hand_right">
-  <link name="right_wrist_yaw_link"/>
+  <link name="right_hand_base"/>
   <xacro:include filename="$(find g1_mujoco_description)/urdf/g1_hands.urdf.xacro"/>
   <xacro:g1_inspire_right_hand_urdf/>

File: g1_mujoco_ros2/g1_mujoco_description/urdf/g1_mujoco.urdf.xacro (robot description, xacro)
@@ -7,4 +7,22 @@
   <xacro:include filename="$(find g1_mujoco_description)/urdf/g1_hands.urdf.xacro"/>
   <xacro:include filename="$(find g1_mujoco_description)/urdf/g1.ros2_control.xacro"/>
+  <link name="world"/>
+  <joint name="world_to_pelvis" type="fixed">
+    <parent link="world"/>
+    <child link="pelvis"/>
+    <origin xyz="0 0 0.793" rpy="0 0 0"/>
+  </joint>
+  <link name="left_hand_base"/>
+  <joint name="left_hand_base_joint" type="fixed">
+    <parent link="left_wrist_yaw_link"/>
+    <child link="left_hand_base"/>
+    <origin xyz="0.05 0 0" rpy="0 -1.57079632679 0"/>
+  </joint>
+  <link name="right_hand_base"/>
+  <joint name="right_hand_base_joint" type="fixed">
+    <parent link="right_wrist_yaw_link"/>
+    <child link="right_hand_base"/>
+    <origin xyz="0.05 0 0" rpy="0 -1.57079632679 0"/>
+  </joint>
   <xacro:g1_optional_hands robot_model="$(arg robot_model)"/>
   <xacro:g1_mujoco_ros2_control

File: rby1_mujoco_ros2/rby1_mujoco_description/urdf/rby1.ros2_control.xacro (robot description, xacro)
@@ -135,10 +135,4 @@
       <xacro:position_joint joint_name="head_1" initial_positions="${initial_positions}"
         include_temperature="${include_temperature}" />
-      <xacro:if value="${robot_model != 'a_wuji' and robot_model != 'm_wuji'}">
-        <xacro:position_joint joint_name="right_trigger" initial_positions="${initial_positions}"
-          include_temperature="${include_temperature}" />
-        <xacro:position_joint joint_name="left_trigger" initial_positions="${initial_positions}"
-          include_temperature="${include_temperature}" />
-      </xacro:if>
       <xacro:if value="${robot_model == 'a_wuji' or robot_model == 'm_wuji'}">
         <xacro:position_joint joint_name="right_finger1_joint1" initial_positions="${initial_positions}" />

File: rby1_mujoco_ros2/rby1_mujoco_description/urdf/rby1.urdf.xacro (robot description, xacro)
@@ -9,6 +9,5 @@
   <xacro:property name="base_robot_model"
     value="${'a' if robot_model == 'a_wuji' else ('m' if robot_model == 'm_wuji' else robot_model)}" />
-  <xacro:property name="gripper_z_offset"
-    value="${0 if base_robot_model == 'a' and robot_version == 'v1.0' else -0.035}" />
+  <xacro:include filename="$(find rby1_mujoco_description)/urdf/wuji_hand/rby1_mount.urdf.xacro" />
   <xacro:if value="${robot_model == 'a_wuji'}">
     <xacro:include filename="$(find rby1_mujoco_description)/urdf/rby1a_wuji/model_v1.2.urdf" />
@@ -24,25 +23,8 @@
   </xacro:if>
   <xacro:if value="${robot_model == 'a_wuji' or robot_model == 'm_wuji'}">
-    <xacro:include filename="$(find rby1_mujoco_description)/urdf/wuji_hand/rby1_mount.urdf.xacro" />
     <xacro:rby1_wuji_hand_mounts />
   </xacro:if>
-  <!-- Virtual gripper joints for unified ros2_control interfaces. -->
   <xacro:if value="${robot_model != 'a_wuji' and robot_model != 'm_wuji'}">
-    <link name="right_gripper_link" />
-    <joint name="right_trigger" type="prismatic">
-      <parent link="ee_right" />
-      <child link="right_gripper_link" />
-      <origin xyz="0 0 ${gripper_z_offset}" rpy="0 0 0" />
-      <axis xyz="0 0 1" />
-      <limit lower="0" upper="1" effort="1" velocity="10" />
-    </joint>
-    <link name="left_gripper_link" />
-    <joint name="left_trigger" type="prismatic">
-      <parent link="ee_left" />
-      <child link="left_gripper_link" />
-      <origin xyz="0 0 ${gripper_z_offset}" rpy="0 0 0" />
-      <axis xyz="0 0 1" />
-      <limit lower="0" upper="1" effort="1" velocity="10" />
-    </joint>
+    <xacro:rby1_hand_base_frames />
   </xacro:if>
   <link name="world" />

File: rby1_mujoco_ros2/rby1_mujoco_description/urdf/rby1a/model.urdf (robot description, URDF)
Before this commit: robot RBY1_A, 34 links, 33 joints
Links:
- removed link ee_finger_l1
- removed link ee_finger_l2
- removed link ee_finger_r1
- removed link ee_finger_r2
- link ee_left: mass 0.46704998 -> None; geometry 
- link ee_right: mass 0.46704998 -> None; geometry 
Joints:
- removed joint gripper_finger_l1
- removed joint gripper_finger_l2
- removed joint gripper_finger_r1
- removed joint gripper_finger_r2

File: rby1_mujoco_ros2/rby1_mujoco_description/urdf/rby1a/model_v1.0.urdf (robot description, URDF)
Before this commit: robot RBY1_A_v1.0, 34 links, 33 joints
Links:
- removed link ee_finger_l1
- removed link ee_finger_l2
- removed link ee_finger_r1
- removed link ee_finger_r2
- link ee_left: mass 0.46704998 -> None; geometry 
- link ee_right: mass 0.46704998 -> None; geometry 
Joints:
- removed joint gripper_finger_l1
- removed joint gripper_finger_l2
- removed joint gripper_finger_r1
- removed joint gripper_finger_r2

File: rby1_mujoco_ros2/rby1_mujoco_description/urdf/rby1a/model_v1.1.urdf (robot description, URDF)
Before this commit: robot RBY1_A_v1.1, 32 links, 31 joints
Links:
- removed link ee_finger_l1
- removed link ee_finger_l2
- removed link ee_finger_r1
- removed link ee_finger_r2
- link ee_left: mass 0.46704998 -> None; geometry 
- link ee_right: mass 0.46704998 -> None; geometry 
Joints:
- removed joint gripper_finger_l1
- removed joint gripper_finger_l2
- removed joint gripper_finger_r1
- removed joint gripper_finger_r2

File: rby1_mujoco_ros2/rby1_mujoco_description/urdf/rby1a/model_v1.2.urdf (robot description, URDF)
Before this commit: robot RBY1_A_v1.2, 32 links, 31 joints
Links:
- removed link ee_finger_l1
- removed link ee_finger_l2
- removed link ee_finger_r1
- removed link ee_finger_r2
- link ee_left: mass 0.46704998 -> None; geometry 
- link ee_right: mass 0.46704998 -> None; geometry 
Joints:
- removed joint gripper_finger_l1
- removed joint gripper_finger_l2
- removed joint gripper_finger_r1
- removed joint gripper_finger_r2

File: rby1_mujoco_ros2/rby1_mujoco_description/urdf/rby1a_wuji/model_v1.2.urdf (robot description, URDF)
Before this commit: robot rby1a_v1.2_wuji, 32 links, 31 joints
Links:
- removed link ee_finger_l1
- removed link ee_finger_l2
- removed link ee_finger_r1
- removed link ee_finger_r2
- link ee_left: mass 0.46704998 -> None
- link ee_right: mass 0.46704998 -> None
Joints:
- removed joint gripper_finger_l1
- removed joint gripper_finger_l2
- removed joint gripper_finger_r1
- removed joint gripper_finger_r2

File: rby1_mujoco_ros2/rby1_mujoco_description/urdf/rby1m/model.urdf (robot description, URDF)
Before this commit: robot RBY1_M, 36 links, 35 joints
Links:
- removed link ee_finger_l1
- removed link ee_finger_l2
- removed link ee_finger_r1
- removed link ee_finger_r2
- link ee_left: mass 0.46704998 -> None; geometry 
- link ee_right: mass 0.46704998 -> None; geometry 
Joints:
- removed joint gripper_finger_l1
- removed joint gripper_finger_l2
- removed joint gripper_finger_r1
- removed joint gripper_finger_r2

File: rby1_mujoco_ros2/rby1_mujoco_description/urdf/rby1m/model_v1.0.urdf (robot description, URDF)
Before this commit: robot RBY1_M_v1.0, 36 links, 35 joints
Links:
- removed link ee_finger_l1
- removed link ee_finger_l2
- removed link ee_finger_r1
- removed link ee_finger_r2
- link ee_left: mass 0.46704998 -> None; geometry 
- link ee_right: mass 0.46704998 -> None; geometry 
Joints:
- removed joint gripper_finger_l1
- removed joint gripper_finger_l2
- removed joint gripper_finger_r1
- removed joint gripper_finger_r2

File: rby1_mujoco_ros2/rby1_mujoco_description/urdf/rby1m/model_v1.1.urdf (robot description, URDF)
Before this commit: robot RBY1_M_v1.1, 34 links, 33 joints
Links:
- removed link ee_finger_l1
- removed link ee_finger_l2
- removed link ee_finger_r1
- removed link ee_finger_r2
- link ee_left: mass 0.46704998 -> None; geometry 
- link ee_right: mass 0.46704998 -> None; geometry 
Joints:
- removed joint gripper_finger_l1
- removed joint gripper_finger_l2
- removed joint gripper_finger_r1
- removed joint gripper_finger_r2

File: rby1_mujoco_ros2/rby1_mujoco_description/urdf/rby1m/model_v1.2.urdf (robot description, URDF)
Before this commit: robot RBY1_M_v1.2, 34 links, 33 joints
Links:
- removed link ee_finger_l1
- removed link ee_finger_l2
- removed link ee_finger_r1
- removed link ee_finger_r2
- link ee_left: mass 0.46704998 -> None; geometry 
- link ee_right: mass 0.46704998 -> None; geometry 
Joints:
- removed joint gripper_finger_l1
- removed joint gripper_finger_l2
- removed joint gripper_finger_r1
- removed joint gripper_finger_r2

File: rby1_mujoco_ros2/rby1_mujoco_description/urdf/rby1m/model_v1.3.urdf (robot description, URDF)
Before this commit: robot RBY1_M_v1.3, 34 links, 33 joints
Links:
- removed link ee_finger_l1
- removed link ee_finger_l2
- removed link ee_finger_r1
- removed link ee_finger_r2
- link ee_left: mass 0.47470074 -> None; geometry 
- link ee_right: mass 0.47470074 -> None; geometry 
Joints:
- removed joint gripper_finger_l1
- removed joint gripper_finger_l2
- removed joint gripper_finger_r1
- removed joint gripper_finger_r2

File: rby1_mujoco_ros2/rby1_mujoco_description/urdf/rby1m_wuji/model_v1.2.urdf (robot description, URDF)
Before this commit: robot RBY1_M_v1.2, 34 links, 33 joints
Links:
- removed link ee_finger_l1
- removed link ee_finger_l2
- removed link ee_finger_r1
- removed link ee_finger_r2
- link ee_left: mass 0.46704998 -> None
- link ee_right: mass 0.46704998 -> None
Joints:
- removed joint gripper_finger_l1
- removed joint gripper_finger_l2
- removed joint gripper_finger_r1
- removed joint gripper_finger_r2
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