Commit message: refactor(menagerie): consolidate hand variant descriptions
- add versioned RBY1 Wuji MJCF variants and update launch description routing
- align G1/Inspire and RBY1/Wuji hand mount frames for simulation and RViz
- prune stale AI Worker bg2 revision assets and duplicated RBY1 Wuji URDFs

File: ai_worker_mujoco_ros2/ai_worker_mujoco_description/urdf/ffw_sg2_rev1_follower/ffw_sg2_follower.urdf.xacro (robot description, xacro)
@@ -145,5 +145,5 @@
     </visual>
   </link>
-  <joint name="$(arg prefix)left_wheel_steer" type="revolute">
+  <joint name="$(arg prefix)left_wheel_steer_joint" type="revolute">
       <parent link="$(arg prefix)base_link"/>
       <child link="$(arg prefix)left_wheel_steer_link"/>
@@ -176,5 +176,5 @@
     </inertial>
   </link>
-  <joint name="$(arg prefix)left_wheel_drive" type="continuous">
+  <joint name="$(arg prefix)left_wheel_drive_joint" type="continuous">
       <parent link="$(arg prefix)left_wheel_steer_link"/>
       <child link="$(arg prefix)left_wheel_drive_link"/>
@@ -213,5 +213,5 @@
     </inertial>
   </link>
-  <joint name="$(arg prefix)right_wheel_steer" type="revolute">
+  <joint name="$(arg prefix)right_wheel_steer_joint" type="revolute">
       <parent link="$(arg prefix)base_link"/>
       <child link="$(arg prefix)right_wheel_steer_link"/>
@@ -244,5 +244,5 @@
     </inertial>
   </link>
-  <joint name="$(arg prefix)right_wheel_drive" type="continuous">
+  <joint name="$(arg prefix)right_wheel_drive_joint" type="continuous">
       <parent link="$(arg prefix)right_wheel_steer_link"/>
       <child link="$(arg prefix)right_wheel_drive_link"/>
@@ -281,5 +281,5 @@
     </inertial>
   </link>
-  <joint name="$(arg prefix)rear_wheel_steer" type="revolute">
+  <joint name="$(arg prefix)rear_wheel_steer_joint" type="revolute">
       <parent link="$(arg prefix)base_link"/>
       <child link="$(arg prefix)rear_wheel_steer_link"/>
@@ -312,5 +312,5 @@
     </inertial>
   </link>
-  <joint name="$(arg prefix)rear_wheel_drive" type="continuous">
+  <joint name="$(arg prefix)rear_wheel_drive_joint" type="continuous">
       <parent link="$(arg prefix)rear_wheel_steer_link"/>
       <child link="$(arg prefix)rear_wheel_drive_link"/>

File: ai_worker_mujoco_ros2/ai_worker_mujoco_description/urdf/ffw_sh5_rev1_follower/ffw_sh5_follower.urdf.xacro (robot description, xacro)
@@ -92,5 +92,5 @@
     <origin xyz="0 0 -0.078" rpy="0 3.14159265359 -1.5708"/>
   </xacro:hx5_d20_right>
-  <joint name="$(arg prefix)left_wheel_steer" type="revolute">
+  <joint name="$(arg prefix)left_wheel_steer_joint" type="revolute">
       <parent link="$(arg prefix)base_link"/>
       <child link="$(arg prefix)left_wheel_steer_link"/>
@@ -123,5 +123,5 @@
     </inertial>
   </link>
-  <joint name="$(arg prefix)left_wheel_drive" type="continuous">
+  <joint name="$(arg prefix)left_wheel_drive_joint" type="continuous">
       <parent link="$(arg prefix)left_wheel_steer_link"/>
       <child link="$(arg prefix)left_wheel_drive_link"/>
@@ -160,5 +160,5 @@
     </inertial>
   </link>
-  <joint name="$(arg prefix)right_wheel_steer" type="revolute">
+  <joint name="$(arg prefix)right_wheel_steer_joint" type="revolute">
       <parent link="$(arg prefix)base_link"/>
       <child link="$(arg prefix)right_wheel_steer_link"/>
@@ -191,5 +191,5 @@
     </inertial>
   </link>
-  <joint name="$(arg prefix)right_wheel_drive" type="continuous">
+  <joint name="$(arg prefix)right_wheel_drive_joint" type="continuous">
       <parent link="$(arg prefix)right_wheel_steer_link"/>
       <child link="$(arg prefix)right_wheel_drive_link"/>
@@ -228,5 +228,5 @@
     </inertial>
   </link>
-  <joint name="$(arg prefix)rear_wheel_steer" type="revolute">
+  <joint name="$(arg prefix)rear_wheel_steer_joint" type="revolute">
       <parent link="$(arg prefix)base_link"/>
       <child link="$(arg prefix)rear_wheel_steer_link"/>
@@ -259,5 +259,5 @@
     </inertial>
   </link>
-  <joint name="$(arg prefix)rear_wheel_drive" type="continuous">
+  <joint name="$(arg prefix)rear_wheel_drive_joint" type="continuous">
       <parent link="$(arg prefix)rear_wheel_steer_link"/>
       <child link="$(arg prefix)rear_wheel_drive_link"/>

File: g1_mujoco_ros2/g1_mujoco_description/urdf/g1_hand_left.urdf.xacro (robot description, xacro)
@@ -1,4 +1,7 @@
 <?xml version="1.0"?>
 <robot xmlns:xacro="http://www.ros.org/wiki/xacro" name="g1_hand_left">
+  <material name="white">
+    <color rgba="0.8 0.8 0.8 1.0"/>
+  </material>
   <link name="left_hand_base"/>
   <xacro:include filename="$(find g1_mujoco_description)/urdf/g1_hands.urdf.xacro"/>

File: g1_mujoco_ros2/g1_mujoco_description/urdf/g1_hand_right.urdf.xacro (robot description, xacro)
@@ -1,4 +1,7 @@
 <?xml version="1.0"?>
 <robot xmlns:xacro="http://www.ros.org/wiki/xacro" name="g1_hand_right">
+  <material name="white">
+    <color rgba="0.8 0.8 0.8 1.0"/>
+  </material>
   <link name="right_hand_base"/>
   <xacro:include filename="$(find g1_mujoco_description)/urdf/g1_hands.urdf.xacro"/>

File: g1_mujoco_ros2/g1_mujoco_description/urdf/g1_hands.urdf.xacro (robot description, xacro)
@@ -187,5 +187,5 @@
       parent="left_hand_base"
       mount_xyz="0 0 0"
-      mount_rpy="0 0 0"/>
+      mount_rpy="0 3.14159265359 1.57079632679"/>
   </xacro:macro>
   <xacro:macro name="g1_inspire_right_hand_urdf">
@@ -193,5 +193,5 @@
       parent="right_hand_base"
       mount_xyz="0 0 0"
-      mount_rpy="0 0 0"/>
+      mount_rpy="0 3.14159265359 -1.57079632679"/>
   </xacro:macro>
   <xacro:macro name="g1_optional_hands" params="robot_model">

File: rby1_mujoco_ros2/rby1_mujoco_description/urdf/rby1.ros2_control.xacro (robot description, xacro)
@@ -52,8 +52,8 @@
         <plugin>mujoco_ros2_control/MujocoSystemInterface</plugin>
         <xacro:if value="${robot_model == 'a_wuji'}">
-          <param name="mujoco_model">$(find rby1_mujoco_description)/mjcf/rby1a/model_act_v1.2_wuji.xml</param>
+          <param name="mujoco_model">$(find rby1_mujoco_description)/mjcf/rby1a/model_act_${robot_version}_wuji.xml</param>
         </xacro:if>
         <xacro:if value="${robot_model == 'm_wuji'}">
-          <param name="mujoco_model">$(find rby1_mujoco_description)/mjcf/rby1m/model_act_v1.2_wuji.xml</param>
+          <param name="mujoco_model">$(find rby1_mujoco_description)/mjcf/rby1m/model_act_${robot_version}_wuji.xml</param>
         </xacro:if>
         <xacro:if value="${(base_robot_model == 'a' or base_robot_model == 'm') and robot_model != 'a_wuji' and robot_model != 'm_wuji'}">

File: rby1_mujoco_ros2/rby1_mujoco_description/urdf/rby1.urdf.xacro (robot description, xacro)
@@ -5,4 +5,5 @@
   <xacro:arg name="initial_positions_file"
     default="$(find rby1_mujoco_description)/config/initial_positions/rby1$(arg robot_model).yaml" />
+  <xacro:arg name="hand_base_offset_z" default="0" />
   <xacro:property name="robot_model" value="$(arg robot_model)" />
   <xacro:property name="robot_version" value="$(arg robot_version)" />
@@ -10,21 +11,15 @@
     value="${'a' if robot_model == 'a_wuji' else ('m' if robot_model == 'm_wuji' else robot_model)}" />
   <xacro:include filename="$(find rby1_mujoco_description)/urdf/wuji_hand/rby1_mount.urdf.xacro" />
-  <xacro:if value="${robot_model == 'a_wuji'}">
-    <xacro:include filename="$(find rby1_mujoco_description)/urdf/rby1a_wuji/model_v1.2.urdf" />
-  </xacro:if>
-  <xacro:if value="${robot_model == 'm_wuji'}">
-    <xacro:include filename="$(find rby1_mujoco_description)/urdf/rby1m_wuji/model_v1.2.urdf" />
-  </xacro:if>
-  <xacro:if value="${base_robot_model == 'a' and robot_model != 'a_wuji'}">
+  <xacro:if value="${base_robot_model == 'a'}">
     <xacro:include filename="$(find rby1_mujoco_description)/urdf/rby1a/model_${robot_version}.urdf" />
   </xacro:if>
-  <xacro:if value="${base_robot_model == 'm' and robot_model != 'm_wuji'}">
+  <xacro:if value="${base_robot_model == 'm'}">
     <xacro:include filename="$(find rby1_mujoco_description)/urdf/rby1m/model_${robot_version}.urdf" />
   </xacro:if>
   <xacro:if value="${robot_model == 'a_wuji' or robot_model == 'm_wuji'}">
-    <xacro:rby1_wuji_hand_mounts />
+    <xacro:rby1_wuji_hand_mounts robot_model="${robot_model}" robot_version="${robot_version}" />
   </xacro:if>
   <xacro:if value="${robot_model != 'a_wuji' and robot_model != 'm_wuji'}">
-    <xacro:rby1_hand_base_frames />
+    <xacro:rby1_hand_base_frames hand_base_offset_z="$(arg hand_base_offset_z)" />
   </xacro:if>
   <link name="world" />

File: rby1_mujoco_ros2/rby1_mujoco_description/urdf/wuji_hand/rby1_mount.urdf.xacro (robot description, xacro)
@@ -1,10 +1,10 @@
 <?xml version="1.0"?>
 <robot xmlns:xacro="http://www.ros.org/wiki/xacro">
-  <xacro:macro name="rby1_hand_base_frames">
+  <xacro:macro name="rby1_hand_base_frames" params="hand_base_offset_z:=0">
     <link name="right_hand_base" />
     <joint name="right_hand_base_joint" type="fixed">
       <parent link="ee_right" />
       <child link="right_hand_base" />
-      <origin xyz="0 0 0" rpy="0 0 0" />
+      <origin xyz="0 0 ${hand_base_offset_z}" rpy="0 0 0" />
     </joint>
     <link name="left_hand_base" />
@@ -12,8 +12,8 @@
       <parent link="ee_left" />
       <child link="left_hand_base" />
-      <origin xyz="0 0 0" rpy="0 0 0" />
+      <origin xyz="0 0 ${hand_base_offset_z}" rpy="0 0 0" />
     </joint>
   </xacro:macro>
-  <xacro:macro name="rby1_wuji_hand_mounts">
+  <xacro:macro name="rby1_wuji_hand_mounts" params="robot_model robot_version">
     <xacro:include
       filename="$(find rby1_mujoco_description)/urdf/wuji_hand/right_with_docking.urdf.xacro" />
@@ -23,10 +23,14 @@
       <parent link="ee_right" />
       <child link="right_hand_base" />
-      <origin xyz="0 0 0" rpy="0 0 0" />
+      <origin
+        xyz="${'0 0 0.066384' if robot_model == 'm_wuji' and robot_version == 'v1.3' else '0 0 0'}"
+        rpy="0 0 0" />
     </joint>
     <joint name="left_hand_base_joint" type="fixed">
       <parent link="ee_left" />
       <child link="left_hand_base" />
-      <origin xyz="0 0 0" rpy="0 0 0" />
+      <origin
+        xyz="${'0 0 0.066384' if robot_model == 'm_wuji' and robot_version == 'v1.3' else '0 0 0'}"
+        rpy="0 0 0" />
     </joint>
   </xacro:macro>
