Commit message: fix(tf): normalize simulation root frame ownership
Remove model-owned world joints, publish explicit map-root transforms from bringup, and keep mobile-base odometry frames unprefixed.

File: ai_worker_mujoco_ros2/ai_worker_mujoco_description/urdf/ffw_bg2_rev4_follower/ffw_bg2_follower.urdf.xacro (robot description, xacro)
@@ -7,10 +7,4 @@
   <xacro:include filename="$(find ai_worker_mujoco_description)/urdf/common/follower/ffw_follower_body.xacro" />
   <xacro:include filename="$(find ai_worker_mujoco_description)/urdf/common/rh_p12_rn_a/rh_p12_rn_a.urdf.xacro" />
-  <link name="world"/>
-  <joint name="$(arg prefix)world_fixed" type="fixed">
-    <parent link="world"/>
-    <child link="$(arg prefix)base_link"/>
-    <origin xyz="0.0 0.0 0.0" rpy="0 0 0"/>
-  </joint>
   <link name="$(arg prefix)base_link">
     <visual>

File: ai_worker_mujoco_ros2/ai_worker_mujoco_description/urdf/ffw_bh5_rev1_follower/ffw_bh5_follower.urdf.xacro (robot description, xacro)
@@ -9,10 +9,4 @@
   <xacro:include filename="$(find ai_worker_mujoco_description)/urdf/common/hx5_d20/hx5_d20_right.urdf.xacro" />
   <!-- Reuse the proven BH5 upper-body ros2_control definition for BH5. -->
-  <link name="world"/>
-  <joint name="$(arg prefix)world_fixed" type="fixed">
-    <parent link="world"/>
-    <child link="$(arg prefix)base_link"/>
-    <origin xyz="0.0 0.0 0.0" rpy="0 0 0"/>
-  </joint>
   <link name="$(arg prefix)base_link">
     <visual>

File: g1_mujoco_ros2/g1_mujoco_description/urdf/g1_mujoco.urdf.xacro (robot description, xacro)
@@ -7,10 +7,4 @@
   <xacro:include filename="$(find g1_mujoco_description)/urdf/g1_hands.urdf.xacro"/>
   <xacro:include filename="$(find g1_mujoco_description)/urdf/g1.ros2_control.xacro"/>
-  <link name="world"/>
-  <joint name="world_to_pelvis" type="fixed">
-    <parent link="world"/>
-    <child link="pelvis"/>
-    <origin xyz="0 0 0.793" rpy="0 0 0"/>
-  </joint>
   <link name="left_hand_base"/>
   <joint name="left_hand_base_joint" type="fixed">

File: rby1_mujoco_ros2/rby1_mujoco_description/urdf/rby1.urdf.xacro (robot description, xacro)
@@ -23,10 +23,4 @@
     <xacro:rby1_hand_base_frames hand_base_offset_z="$(arg hand_base_offset_z)" />
   </xacro:if>
-  <link name="world" />
-  <joint name="world_to_base" type="planar">
-    <parent link="world" />
-    <child link="base" />
-    <origin xyz="0 0 0" rpy="0 0 0" />
-  </joint>
   <!-- ros2_control -->
   <xacro:include filename="$(find rby1_mujoco_description)/urdf/rby1.ros2_control.xacro" />
