Commit message: fix(rby1): align mobile wheel velocity limits
Set A-series wheel actuator limits to 15 rad/s and M-series limits to 19.7 rad/s across supported model variants. Align M-series URDF wheel limits with the simulator actuator limits.

File: rby1_mujoco_ros2/rby1_mujoco_description/urdf/rby1m/model.urdf (robot description, URDF)
Before this commit: robot RBY1_M, 32 links, 31 joints
Joints:
- joint wheel_fl: limit effort=100 velocity=100 -> effort=100 velocity=19.7
- joint wheel_fr: limit effort=100 velocity=100 -> effort=100 velocity=19.7
- joint wheel_rl: limit effort=100 velocity=100 -> effort=100 velocity=19.7
- joint wheel_rr: limit effort=100 velocity=100 -> effort=100 velocity=19.7

File: rby1_mujoco_ros2/rby1_mujoco_description/urdf/rby1m/model_v1.0.urdf (robot description, URDF)
Before this commit: robot RBY1_M_v1.0, 32 links, 31 joints
Joints:
- joint wheel_fl: limit effort=100 velocity=100 -> effort=100 velocity=19.7
- joint wheel_fr: limit effort=100 velocity=100 -> effort=100 velocity=19.7
- joint wheel_rl: limit effort=100 velocity=100 -> effort=100 velocity=19.7
- joint wheel_rr: limit effort=100 velocity=100 -> effort=100 velocity=19.7

File: rby1_mujoco_ros2/rby1_mujoco_description/urdf/rby1m/model_v1.1.urdf (robot description, URDF)
Before this commit: robot RBY1_M_v1.1, 30 links, 29 joints
Joints:
- joint wheel_fl: limit effort=100 velocity=100 -> effort=100 velocity=19.7
- joint wheel_fr: limit effort=100 velocity=100 -> effort=100 velocity=19.7
- joint wheel_rl: limit effort=100 velocity=100 -> effort=100 velocity=19.7
- joint wheel_rr: limit effort=100 velocity=100 -> effort=100 velocity=19.7

File: rby1_mujoco_ros2/rby1_mujoco_description/urdf/rby1m/model_v1.2.urdf (robot description, URDF)
Before this commit: robot RBY1_M_v1.2, 30 links, 29 joints
Joints:
- joint wheel_fl: limit effort=100 velocity=100 -> effort=100 velocity=19.7
- joint wheel_fr: limit effort=100 velocity=100 -> effort=100 velocity=19.7
- joint wheel_rl: limit effort=100 velocity=100 -> effort=100 velocity=19.7
- joint wheel_rr: limit effort=100 velocity=100 -> effort=100 velocity=19.7

File: rby1_mujoco_ros2/rby1_mujoco_description/urdf/rby1m/model_v1.3.urdf (robot description, URDF)
Before this commit: robot RBY1_M_v1.3, 30 links, 29 joints
Joints:
- joint wheel_fl: limit effort=100 velocity=100 -> effort=100 velocity=19.7
- joint wheel_fr: limit effort=100 velocity=100 -> effort=100 velocity=19.7
- joint wheel_rl: limit effort=100 velocity=100 -> effort=100 velocity=19.7
- joint wheel_rr: limit effort=100 velocity=100 -> effort=100 velocity=19.7
