Commit message: fix(description): synchronize versioned RBY1 model properties
- align A and M inertial data and joint limits with versioned robot models
- propagate the same body properties to Wuji-equipped MJCF variants
- standardize M wheel velocity limits across supported versions

File: rby1_mujoco_ros2/rby1_mujoco_description/urdf/rby1m/model_v1.0.urdf (robot description, URDF)
Before this commit: robot RBY1_M_v1.0, 32 links, 31 joints
Joints:
- joint wheel_fl: limit effort=100 velocity=19.7 -> effort=100 velocity=15.707963268
- joint wheel_fr: limit effort=100 velocity=19.7 -> effort=100 velocity=15.707963268
- joint wheel_rl: limit effort=100 velocity=19.7 -> effort=100 velocity=15.707963268
- joint wheel_rr: limit effort=100 velocity=19.7 -> effort=100 velocity=15.707963268

File: rby1_mujoco_ros2/rby1_mujoco_description/urdf/rby1m/model_v1.1.urdf (robot description, URDF)
Before this commit: robot RBY1_M_v1.1, 30 links, 29 joints
Joints:
- joint wheel_fl: limit effort=100 velocity=19.7 -> effort=100 velocity=15.707963268
- joint wheel_fr: limit effort=100 velocity=19.7 -> effort=100 velocity=15.707963268
- joint wheel_rl: limit effort=100 velocity=19.7 -> effort=100 velocity=15.707963268
- joint wheel_rr: limit effort=100 velocity=19.7 -> effort=100 velocity=15.707963268

File: rby1_mujoco_ros2/rby1_mujoco_description/urdf/rby1m/model_v1.2.urdf (robot description, URDF)
Before this commit: robot RBY1_M_v1.2, 30 links, 29 joints
Joints:
- joint wheel_fl: limit effort=100 velocity=19.7 -> effort=100 velocity=15.707963268
- joint wheel_fr: limit effort=100 velocity=19.7 -> effort=100 velocity=15.707963268
- joint wheel_rl: limit effort=100 velocity=19.7 -> effort=100 velocity=15.707963268
- joint wheel_rr: limit effort=100 velocity=19.7 -> effort=100 velocity=15.707963268

File: rby1_mujoco_ros2/rby1_mujoco_description/urdf/rby1m/model_v1.3.urdf (robot description, URDF)
Before this commit: robot RBY1_M_v1.3, 30 links, 29 joints
Joints:
- joint wheel_fl: limit effort=100 velocity=19.7 -> effort=100 velocity=15.707963268
- joint wheel_fr: limit effort=100 velocity=19.7 -> effort=100 velocity=15.707963268
- joint wheel_rl: limit effort=100 velocity=19.7 -> effort=100 velocity=15.707963268
- joint wheel_rr: limit effort=100 velocity=19.7 -> effort=100 velocity=15.707963268
