Commit message: Refactor base link naming across MJCF and URDF files
- Changed the name of the "base" body/link to "base_link" in multiple MJCF files (rby1_v1.0.xml, rby1_v1.1.xml, rby1_v1.2.xml, rby1_v1.3.xml, and their respective wuji variants) to maintain consistency.
- Updated the base link name in the base.xml asset file.
- Modified the URDF files (model.urdf, model_v1.0.urdf, model_v1.1.urdf, model_v1.2.urdf, model_v1.3.urdf) to reflect the new base link name.
- Adjusted the robot_base_frame parameter in the navigation configuration files (rby1a.yaml and rby1m.yaml) to use "base_link" instead of "base".

File: rby1_mujoco_ros2/rby1_mujoco_description/urdf/rby1a/model.urdf (robot description, URDF)
Before this commit: robot RBY1_A, 30 links, 29 joints
Links:
- removed link base
- added link base_link, mass 60.08042639; visual mesh filename=package://rby1_mujoco_description/meshes/rby1a/base.dae
Joints:
- joint left_wheel: parent base -> base_link
- joint right_wheel: parent base -> base_link
- joint torso_0: parent base -> base_link

File: rby1_mujoco_ros2/rby1_mujoco_description/urdf/rby1a/model_v1.0.urdf (robot description, URDF)
Before this commit: robot RBY1_A_v1.0, 30 links, 29 joints
Links:
- removed link base
- added link base_link, mass 60.08042639; visual mesh filename=package://rby1_mujoco_description/meshes/rby1a/base.dae
Joints:
- joint left_wheel: parent base -> base_link
- joint right_wheel: parent base -> base_link
- joint torso_0: parent base -> base_link

File: rby1_mujoco_ros2/rby1_mujoco_description/urdf/rby1a/model_v1.1.urdf (robot description, URDF)
Before this commit: robot RBY1_A_v1.1, 28 links, 27 joints
Links:
- removed link base
- added link base_link, mass 60.08042639; visual mesh filename=package://rby1_mujoco_description/meshes/rby1a/base.dae
Joints:
- joint left_wheel: parent base -> base_link
- joint right_wheel: parent base -> base_link
- joint torso_0: parent base -> base_link

File: rby1_mujoco_ros2/rby1_mujoco_description/urdf/rby1a/model_v1.2.urdf (robot description, URDF)
Before this commit: robot RBY1_A_v1.2, 28 links, 27 joints
Links:
- removed link base
- added link base_link, mass 60.08042639; visual mesh filename=package://rby1_mujoco_description/meshes/rby1a/base.dae
Joints:
- joint left_wheel: parent base -> base_link
- joint right_wheel: parent base -> base_link
- joint torso_0: parent base -> base_link

File: rby1_mujoco_ros2/rby1_mujoco_description/urdf/rby1m/model.urdf (robot description, URDF)
Before this commit: robot RBY1_M, 32 links, 31 joints
Links:
- removed link base
- added link base_link, mass 82.93082168; visual mesh filename=package://rby1_mujoco_description/meshes/rby1m/base.dae
Joints:
- joint torso_0: parent base -> base_link
- joint wheel_fl: parent base -> base_link
- joint wheel_fr: parent base -> base_link
- joint wheel_rl: parent base -> base_link
- joint wheel_rr: parent base -> base_link

File: rby1_mujoco_ros2/rby1_mujoco_description/urdf/rby1m/model_v1.0.urdf (robot description, URDF)
Before this commit: robot RBY1_M_v1.0, 32 links, 31 joints
Links:
- removed link base
- added link base_link, mass 82.93082168; visual mesh filename=package://rby1_mujoco_description/meshes/rby1m/base.dae
Joints:
- joint torso_0: parent base -> base_link
- joint wheel_fl: parent base -> base_link
- joint wheel_fr: parent base -> base_link
- joint wheel_rl: parent base -> base_link
- joint wheel_rr: parent base -> base_link

File: rby1_mujoco_ros2/rby1_mujoco_description/urdf/rby1m/model_v1.1.urdf (robot description, URDF)
Before this commit: robot RBY1_M_v1.1, 30 links, 29 joints
Links:
- removed link base
- added link base_link, mass 82.93082168; visual mesh filename=package://rby1_mujoco_description/meshes/rby1m/base.dae
Joints:
- joint torso_0: parent base -> base_link
- joint wheel_fl: parent base -> base_link
- joint wheel_fr: parent base -> base_link
- joint wheel_rl: parent base -> base_link
- joint wheel_rr: parent base -> base_link

File: rby1_mujoco_ros2/rby1_mujoco_description/urdf/rby1m/model_v1.2.urdf (robot description, URDF)
Before this commit: robot RBY1_M_v1.2, 30 links, 29 joints
Links:
- removed link base
- added link base_link, mass 82.93082168; visual mesh filename=package://rby1_mujoco_description/meshes/rby1m/base.dae
Joints:
- joint torso_0: parent base -> base_link
- joint wheel_fl: parent base -> base_link
- joint wheel_fr: parent base -> base_link
- joint wheel_rl: parent base -> base_link
- joint wheel_rr: parent base -> base_link

File: rby1_mujoco_ros2/rby1_mujoco_description/urdf/rby1m/model_v1.3.urdf (robot description, URDF)
Before this commit: robot RBY1_M_v1.3, 30 links, 29 joints
Links:
- removed link base
- added link base_link, mass 82.93082168; visual mesh filename=package://rby1_mujoco_description/meshes/rby1m/base.dae
Joints:
- joint torso_0: parent base -> base_link
- joint wheel_fl: parent base -> base_link
- joint wheel_fr: parent base -> base_link
- joint wheel_rl: parent base -> base_link
- joint wheel_rr: parent base -> base_link
