Commit message: feat: update collision geometries and origins for RBY1 models

File: rby1_mujoco_ros2/rby1_mujoco_description/urdf/rby1a/model_v1.0.urdf (robot description, URDF)
Before this commit: robot RBY1_A_v1.0, 30 links, 29 joints
Links:
- link base_link: geometry collision box size=0.64 0.52 0.22; visual mesh filename=package://rby1_mujoco_description/meshes/rby1a/base.dae
- link link_head_0: geometry collision sphere radius=0.07; visual mesh filename=package://rby1_mujoco_description/meshes/rby1a/PAN_TILT_1.d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
- link link_left_arm_5: geometry collision cylinder length=0.325 radius=0.075; visual mesh filename=package://rby1_mujoco_description/meshes/rby1a/LINK_19.dae
- link link_right_arm_5: geometry collision cylinder length=0.325 radius=0.075; visual mesh filename=package://rby1_mujoco_description/meshes/rby1a/LINK_12.dae

File: rby1_mujoco_ros2/rby1_mujoco_description/urdf/rby1a/model_v1.1.urdf (robot description, URDF)
Before this commit: robot RBY1_A_v1.1, 28 links, 27 joints
Links:
- link base_link: geometry collision box size=0.64 0.52 0.22; visual mesh filename=package://rby1_mujoco_description/meshes/rby1a/base.dae
- link link_head_0: geometry collision sphere radius=0.07; visual mesh filename=package://rby1_mujoco_description/meshes/rby1a/PAN_TILT_1.d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
- link link_left_arm_5: geometry collision cylinder length=0.325 radius=0.075; visual mesh filename=package://rby1_mujoco_description/meshes/rby1a/LINK_19_v1.1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
- link link_right_arm_5: geometry collision cylinder length=0.325 radius=0.075; visual mesh filename=package://rby1_mujoco_description/meshes/rby1a/LINK_12_v1.1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

File: rby1_mujoco_ros2/rby1_mujoco_description/urdf/rby1a/model_v1.2.urdf (robot description, URDF)
Before this commit: robot RBY1_A_v1.2, 28 links, 27 joints
Links:
- link base_link: geometry collision box size=0.64 0.52 0.22; visual mesh filename=package://rby1_mujoco_description/meshes/rby1a/base.dae
- link link_head_0: geometry collision sphere radius=0.10; visual mesh filename=package://rby1_mujoco_description/meshes/rby1a/NECK_0.dae
- link link_left_arm_5: geometry collision cylinder length=0.325 radius=0.075; visual mesh filename=package://rby1_mujoco_description/meshes/rby1a/LINK_19_v1.1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
- link link_right_arm_5: geometry collision cylinder length=0.325 radius=0.075; visual mesh filename=package://rby1_mujoco_description/meshes/rby1a/LINK_12_v1.1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

File: rby1_mujoco_ros2/rby1_mujoco_description/urdf/rby1m/model_v1.0.urdf (robot description, URDF)
Before this commit: robot RBY1_M_v1.0, 32 links, 31 joints
Links:
- link base_link: geometry collision box size=0.70 0.60 0.22; visual mesh filename=package://rby1_mujoco_description/meshes/rby1m/base.dae
- link link_head_0: geometry collision sphere radius=0.07; visual mesh filename=package://rby1_mujoco_description/meshes/rby1m/PAN_TILT_1.d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
- link link_left_arm_5: geometry collision cylinder length=0.325 radius=0.075; visual mesh filename=package://rby1_mujoco_description/meshes/rby1m/LINK_19.dae
- link link_right_arm_5: geometry collision cylinder length=0.325 radius=0.075; visual mesh filename=package://rby1_mujoco_description/meshes/rby1m/LINK_12.dae

File: rby1_mujoco_ros2/rby1_mujoco_description/urdf/rby1m/model_v1.1.urdf (robot description, URDF)
Before this commit: robot RBY1_M_v1.1, 30 links, 29 joints
Links:
- link base_link: geometry collision box size=0.70 0.60 0.22; visual mesh filename=package://rby1_mujoco_description/meshes/rby1m/base.dae
- link link_head_0: geometry collision sphere radius=0.07; visual mesh filename=package://rby1_mujoco_description/meshes/rby1m/PAN_TILT_1.d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
- link link_left_arm_5: geometry collision cylinder length=0.325 radius=0.075; visual mesh filename=package://rby1_mujoco_description/meshes/rby1m/LINK_19_v1.1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
- link link_right_arm_5: geometry collision cylinder length=0.325 radius=0.075; visual mesh filename=package://rby1_mujoco_description/meshes/rby1m/LINK_12_v1.1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

File: rby1_mujoco_ros2/rby1_mujoco_description/urdf/rby1m/model_v1.2.urdf (robot description, URDF)
Before this commit: robot RBY1_M_v1.2, 30 links, 29 joints
Links:
- link base_link: geometry collision box size=0.70 0.60 0.22; visual mesh filename=package://rby1_mujoco_description/meshes/rby1m/base.dae
- link link_head_0: geometry collision sphere radius=0.10; visual mesh filename=package://rby1_mujoco_description/meshes/rby1m/NECK_0.dae
- link link_left_arm_5: geometry collision cylinder length=0.325 radius=0.075; visual mesh filename=package://rby1_mujoco_description/meshes/rby1m/LINK_19_v1.1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
- link link_right_arm_5: geometry collision cylinder length=0.325 radius=0.075; visual mesh filename=package://rby1_mujoco_description/meshes/rby1m/LINK_12_v1.1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

File: rby1_mujoco_ros2/rby1_mujoco_description/urdf/rby1m/model_v1.3.urdf (robot description, URDF)
Before this commit: robot RBY1_M_v1.3, 30 links, 29 joints
Links:
- link base_link: geometry collision box size=0.70 0.60 0.22; visual mesh filename=package://rby1_mujoco_description/meshes/rby1m/base.dae
- link link_head_0: geometry collision sphere radius=0.10; visual mesh filename=package://rby1_mujoco_description/meshes/rby1m/NECK_0.dae
- link link_left_arm_5: geometry collision cylinder length=0.325 radius=0.075; visual mesh filename=package://rby1_mujoco_description/meshes/rby1m/LINK_19_WP.d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
- link link_right_arm_5: geometry collision cylinder length=0.325 radius=0.075; visual mesh filename=package://rby1_mujoco_description/meshes/rby1m/LINK_12_WP.d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
