Commit message: fix(mobile-aloha): align PiPER frame and end-effector geometry
- remove the duplicate yaw transform from the bundled support-frame meshes
- map follower grippers and leader handles into the wrist frame
- verify support contacts and ROS-to-MuJoCo end-effector alignment

File: mobile_aloha_mujoco_ros2/mobile_aloha_mujoco_description/urdf/mobile_aloha_piper.urdf.xacro (robot description, xacro)
@@ -121,36 +121,37 @@
   </link>
   <link name="body_link">
-    <visual>
-      <origin xyz="0 0 0.168" rpy="0 0 ${pi}"/>
+    <!-- The bundled STL parts already include the upstream body's yaw transform. -->
+    <visual>
+      <origin xyz="0 0 0.168"/>
       <geometry><mesh filename="${official_mesh_root}/body_0.STL"/></geometry>
       <material name="body_white"/>
     </visual>
     <visual>
-      <origin xyz="0 0 0.168" rpy="0 0 ${pi}"/>
+      <origin xyz="0 0 0.168"/>
       <geometry><mesh filename="${official_mesh_root}/body_1.STL"/></geometry>
       <material name="body_white"/>
     </visual>
     <visual>
-      <origin xyz="0 0 0.168" rpy="0 0 ${pi}"/>
+      <origin xyz="0 0 0.168"/>
       <geometry><mesh filename="${official_mesh_root}/body_2.STL"/></geometry>
       <material name="body_white"/>
     </visual>
     <visual>
-      <origin xyz="0 0 0.168" rpy="0 0 ${pi}"/>
+      <origin xyz="0 0 0.168"/>
       <geometry><mesh filename="${official_mesh_root}/body_3.STL"/></geometry>
       <material name="body_white"/>
     </visual>
     <visual>
-      <origin xyz="0 0 0.168" rpy="0 0 ${pi}"/>
+      <origin xyz="0 0 0.168"/>
       <geometry><mesh filename="${official_mesh_root}/body_4.STL"/></geometry>
       <material name="body_white"/>
     </visual>
     <visual>
-      <origin xyz="0 0 0.168" rpy="0 0 ${pi}"/>
+      <origin xyz="0 0 0.168"/>
       <geometry><mesh filename="${official_mesh_root}/body_5.STL"/></geometry>
       <material name="body_white"/>
     </visual>
     <visual>
-      <origin xyz="0 0 0.168" rpy="0 0 ${pi}"/>
+      <origin xyz="0 0 0.168"/>
       <geometry><mesh filename="${official_mesh_root}/body_6.STL"/></geometry>
       <material name="body_white"/>
