Commit message: fix(mobile-aloha): align VX300S grippers with MuJoCo
- restore mounting frames, mesh geometry and prismatic finger axes
- check closed/open gripper poses with native URDF and MJCF loaders

File: mobile_aloha_mujoco_ros2/mobile_aloha_mujoco_description/urdf/mobile_aloha.urdf.xacro (robot description, xacro)
@@ -154,20 +154,4 @@
         <inertia ixx="0.0007" ixy="0" ixz="0" iyy="0.0007" iyz="0" izz="0.0005"/>
       </inertial>
-      <visual>
-        <geometry><mesh filename="${mesh_root}/vx300s_7_gripper_prop.stl"/></geometry>
-        <material name="black"/>
-      </visual>
-      <visual>
-        <geometry><mesh filename="${mesh_root}/vx300s_7_gripper_bar.stl"/></geometry>
-        <material name="black"/>
-      </visual>
-      <collision>
-        <origin xyz="0 -0.0023 0.0094" rpy="0 0 0"/>
-        <geometry><box size="0.153 0.069 0.028"/></geometry>
-      </collision>
-      <collision>
-        <origin xyz="0 -0.0121 -0.0208" rpy="0 0 0"/>
-        <geometry><box size="0.032 0.050 0.039"/></geometry>
-      </collision>
     </link>
     <joint name="${prefix}_wrist_rotate" type="revolute">
@@ -179,24 +163,61 @@
       <dynamics damping="1.2"/>
     </joint>
+    <!-- Retain the MuJoCo mounting frame for the rail and both sliding fingers. -->
+    <link name="${prefix}_gripper_base">
+      <visual>
+        <geometry><mesh filename="${mesh_root}/vx300s_7_gripper_prop.stl"/></geometry>
+        <material name="black"/>
+      </visual>
+      <visual>
+        <geometry><mesh filename="${mesh_root}/vx300s_7_gripper_bar.stl"/></geometry>
+        <material name="black"/>
+      </visual>
+      <collision>
+        <geometry><mesh filename="${mesh_root}/vx300s_7_gripper_prop.stl"/></geometry>
+      </collision>
+      <collision>
+        <geometry><mesh filename="${mesh_root}/vx300s_7_gripper_bar.stl"/></geometry>
+      </collision>
+    </link>
+    <joint name="${prefix}_gripper_base_joint" type="fixed">
+      <!-- MJCF intrinsic euler="0 1.57 -1.57", converted to URDF fixed-axis RPY. -->
+      <origin xyz="0.035 0 0" rpy="-1.569999999748 0.000796326542407 -1.570795692658"/>
+      <parent link="${prefix}_gripper_link"/>
+      <child link="${prefix}_gripper_base"/>
+    </joint>
     <link name="${prefix}_left_finger_link">
-      <visual><origin xyz="0.10 0.02 0"/><geometry><box size="0.12 0.015 0.02"/></geometry><material name="black"/></visual>
-      <collision><origin xyz="0.10 0.02 0"/><geometry><box size="0.12 0.015 0.02"/></geometry></collision>
+      <visual>
+        <origin xyz="0.0141637 0.0211727 0.06" rpy="${pi / 2} ${pi / 2} 0"/>
+        <geometry><mesh filename="${mesh_root}/vx300s_8_custom_finger_left.stl"/></geometry>
+        <material name="black"/>
+      </visual>
+      <collision>
+        <origin xyz="0.0141637 0.0211727 0.06" rpy="${pi / 2} ${pi / 2} 0"/>
+        <geometry><mesh filename="${mesh_root}/vx300s_8_custom_finger_left.stl"/></geometry>
+      </collision>
     </link>
     <joint name="${prefix}_left_finger" type="prismatic">
-      <origin xyz="0.035 0 0" rpy="0 0 0"/>
-      <parent link="${prefix}_gripper_link"/>
+      <origin xyz="0.0191 -0.0141637 0.0211727" rpy="${-pi / 2} 0 ${pi / 2}"/>
+      <parent link="${prefix}_gripper_base"/>
       <child link="${prefix}_left_finger_link"/>
-      <axis xyz="0 1 0"/>
+      <axis xyz="0 0 -1"/>
       <limit lower="0.002" upper="0.037" effort="20" velocity="1"/>
     </joint>
     <link name="${prefix}_right_finger_link">
-      <visual><origin xyz="0.10 -0.02 0"/><geometry><box size="0.12 0.015 0.02"/></geometry><material name="black"/></visual>
-      <collision><origin xyz="0.10 -0.02 0"/><geometry><box size="0.12 0.015 0.02"/></geometry></collision>
+      <visual>
+        <origin xyz="0.0141637 -0.0211727 0.0597067" rpy="${-pi / 2} ${-pi / 2} 0"/>
+        <geometry><mesh filename="${mesh_root}/vx300s_8_custom_finger_right.stl"/></geometry>
+        <material name="black"/>
+      </visual>
+      <collision>
+        <origin xyz="0.0141637 -0.0211727 0.0597067" rpy="${-pi / 2} ${-pi / 2} 0"/>
+        <geometry><mesh filename="${mesh_root}/vx300s_8_custom_finger_right.stl"/></geometry>
+      </collision>
     </link>
     <joint name="${prefix}_right_finger" type="prismatic">
-      <origin xyz="0.035 0 0" rpy="0 0 0"/>
-      <parent link="${prefix}_gripper_link"/>
+      <origin xyz="-0.0191 -0.0141637 0.0211727" rpy="${pi / 2} 0 ${pi / 2}"/>
+      <parent link="${prefix}_gripper_base"/>
       <child link="${prefix}_right_finger_link"/>
-      <axis xyz="0 -1 0"/>
+      <axis xyz="0 0 -1"/>
       <limit lower="0.002" upper="0.037" effort="20" velocity="1"/>
       <mimic joint="${prefix}_left_finger" multiplier="1" offset="0"/>
