Commit message: feat(mobile-aloha): expose fixed arm flange frames

File: mobile_aloha_mujoco_ros2/mobile_aloha_mujoco_description/urdf/mobile_aloha_mujoco.urdf.xacro (robot description, xacro)
@@ -5,3 +5,15 @@
   <xacro:include filename="$(find mobile_aloha_mujoco_description)/urdf/mobile_aloha.ros2_control.xacro"/>
   <xacro:mobile_aloha_ros2_control headless="$(arg headless)"/>
+  <link name="left_flange"/>
+  <joint name="left_flange_joint" type="fixed">
+    <origin xyz="0.042825 0 0" rpy="3.141592653589793 -1.570796326794897 0"/>
+    <parent link="left_gripper_link"/>
+    <child link="left_flange"/>
+  </joint>
+  <link name="right_flange"/>
+  <joint name="right_flange_joint" type="fixed">
+    <origin xyz="0.042825 0 0" rpy="3.141592653589793 -1.570796326794897 0"/>
+    <parent link="right_gripper_link"/>
+    <child link="right_flange"/>
+  </joint>
 </robot>

File: mobile_aloha_mujoco_ros2/mobile_aloha_mujoco_description/urdf/mobile_aloha_piper_mujoco.urdf.xacro (robot description, xacro)
@@ -5,3 +5,15 @@
   <xacro:include filename="$(find mobile_aloha_mujoco_description)/urdf/mobile_aloha_piper.ros2_control.xacro"/>
   <xacro:mobile_aloha_piper_ros2_control headless="$(arg headless)"/>
+  <link name="left_flange"/>
+  <joint name="left_flange_joint" type="fixed">
+    <origin xyz="0 0 0" rpy="0 0 1.570796326794897"/>
+    <parent link="fl_link6"/>
+    <child link="left_flange"/>
+  </joint>
+  <link name="right_flange"/>
+  <joint name="right_flange_joint" type="fixed">
+    <origin xyz="0 0 0" rpy="0 0 1.570796326794897"/>
+    <parent link="fr_link6"/>
+    <child link="right_flange"/>
+  </joint>
 </robot>

Commit message: fix(mobile-aloha): align flanges and re-zero PiPER wrists

File: mobile_aloha_mujoco_ros2/mobile_aloha_mujoco_description/urdf/mobile_aloha_mujoco.urdf.xacro (robot description, xacro)
@@ -7,5 +7,5 @@
   <link name="left_flange"/>
   <joint name="left_flange_joint" type="fixed">
-    <origin xyz="0.042825 0 0" rpy="3.141592653589793 -1.570796326794897 0"/>
+    <origin xyz="0.042825 0 0" rpy="0 0 0"/>
     <parent link="left_gripper_link"/>
     <child link="left_flange"/>
@@ -13,5 +13,5 @@
   <link name="right_flange"/>
   <joint name="right_flange_joint" type="fixed">
-    <origin xyz="0.042825 0 0" rpy="3.141592653589793 -1.570796326794897 0"/>
+    <origin xyz="0.042825 0 0" rpy="0 0 0"/>
     <parent link="right_gripper_link"/>
     <child link="right_flange"/>

File: mobile_aloha_mujoco_ros2/mobile_aloha_mujoco_description/urdf/mobile_aloha_piper.ros2_control.xacro (robot description, xacro)
@@ -22,5 +22,5 @@
     <xacro:piper_position_joint name="${prefix}_joint3" initial_value="-1.3485"/>
     <xacro:piper_position_joint name="${prefix}_joint4"/>
-    <xacro:piper_position_joint name="${prefix}_joint5"/>
+    <xacro:piper_position_joint name="${prefix}_joint5" initial_value="-0.0872495900012399"/>
     <xacro:piper_position_joint name="${prefix}_joint6"/>
     <xacro:piper_position_joint name="${prefix}_joint7" initial_value="0.035"/>

File: mobile_aloha_mujoco_ros2/mobile_aloha_mujoco_description/urdf/mobile_aloha_piper.urdf.xacro (robot description, xacro)
@@ -30,4 +30,5 @@
     </link>
   </xacro:macro>
+  <!-- Native joint5 = model joint5 + 0.0872495900012399 rad; model zero has a horizontal tool. -->
   <xacro:macro name="piper" params="prefix parent xyz gripper_prefix finger_origin">
     <xacro:piper_link name="${prefix}_base_link" mesh="base_link.stl"/>
@@ -71,9 +72,9 @@
     <xacro:piper_link name="${prefix}_link5" mesh="link5.stl"/>
     <joint name="${prefix}_joint5" type="revolute">
-      <origin xyz="0 0 0" rpy="1.5708 0 0"/>
+      <origin xyz="0 0 0" rpy="1.570800014025604 -0.08724959000064958 -3.21301354522241e-07"/>
       <parent link="${prefix}_link4"/>
       <child link="${prefix}_link5"/>
       <axis xyz="0 0 1"/>
-      <limit lower="-1.22" upper="1.22" effort="100" velocity="3"/>
+      <limit lower="-1.30724959000124" upper="1.13275040999876" effort="100" velocity="3"/>
     </joint>
     <xacro:piper_link name="${prefix}_link6" mesh="${gripper_prefix}_link6.stl"/>

File: mobile_aloha_mujoco_ros2/mobile_aloha_mujoco_description/urdf/mobile_aloha_piper_mujoco.urdf.xacro (robot description, xacro)
@@ -7,5 +7,5 @@
   <link name="left_flange"/>
   <joint name="left_flange_joint" type="fixed">
-    <origin xyz="0 0 0" rpy="0 0 1.570796326794897"/>
+    <origin xyz="0 0 0" rpy="-1.570796326794897 -1.570796326794897 0"/>
     <parent link="fl_link6"/>
     <child link="left_flange"/>
@@ -13,5 +13,5 @@
   <link name="right_flange"/>
   <joint name="right_flange_joint" type="fixed">
-    <origin xyz="0 0 0" rpy="0 0 1.570796326794897"/>
+    <origin xyz="0 0 0" rpy="-1.570796326794897 -1.570796326794897 0"/>
     <parent link="fr_link6"/>
     <child link="right_flange"/>
