Commit message: fix(rb): prevent servo saturation overshoot and align joint limits

File: rb_mujoco_ros2/rb_mujoco_description/urdf/rb10_1300e.urdf (robot description, URDF)
Before this commit: robot rb10_1300e, 8 links, 7 joints
Joints:
- joint base: limit lower=-3.14 upper=3.14 effort=10 velocity=3.14 -> lower=-6.28318530717959 upper=6.28318530717959 effort=10 velocity=2.0943951023932
- joint elbow: limit lower=-3.14 upper=3.14 effort=10 velocity=3.14 -> lower=-2.87979326579064 upper=2.87979326579064 effort=10 velocity=3.14159265358979
- joint shoulder: limit lower=-3.14 upper=3.14 effort=10 velocity=3.14 -> lower=-6.28318530717959 upper=6.28318530717959 effort=10 velocity=2.0943951023932
- joint wrist1: limit lower=-3.14 upper=3.14 effort=10 velocity=3.14 -> lower=-6.28318530717959 upper=6.28318530717959 effort=10 velocity=3.14159265358979
- joint wrist2: limit lower=-3.14 upper=3.14 effort=10 velocity=3.14 -> lower=-6.28318530717959 upper=6.28318530717959 effort=10 velocity=3.14159265358979
- joint wrist3: limit lower=-3.14 upper=3.14 effort=10 velocity=3.14 -> lower=-6.28318530717959 upper=6.28318530717959 effort=10 velocity=3.14159265358979

File: rb_mujoco_ros2/rb_mujoco_description/urdf/rb10_1300e_u.urdf (robot description, URDF)
Before this commit: robot rb10_1300e_u, 8 links, 7 joints
Joints:
- joint base: limit lower=-3.14 upper=3.14 effort=10 velocity=3.14 -> lower=-6.28318530717959 upper=6.28318530717959 effort=10 velocity=2.0943951023932
- joint elbow: limit lower=-3.14 upper=3.14 effort=10 velocity=3.14 -> lower=-2.87979326579064 upper=2.87979326579064 effort=10 velocity=3.14159265358979
- joint shoulder: limit lower=-3.14 upper=3.14 effort=10 velocity=3.14 -> lower=-6.28318530717959 upper=6.28318530717959 effort=10 velocity=2.0943951023932
- joint wrist1: limit lower=-3.14 upper=3.14 effort=10 velocity=3.14 -> lower=-6.28318530717959 upper=6.28318530717959 effort=10 velocity=3.14159265358979
- joint wrist2: limit lower=-3.14 upper=3.14 effort=10 velocity=3.14 -> lower=-6.28318530717959 upper=6.28318530717959 effort=10 velocity=3.14159265358979
- joint wrist3: limit lower=-3.14 upper=3.14 effort=10 velocity=3.14 -> lower=-6.28318530717959 upper=6.28318530717959 effort=10 velocity=3.14159265358979

File: rb_mujoco_ros2/rb_mujoco_description/urdf/rb16_900e.urdf (robot description, URDF)
Before this commit: robot rb16_900e, 8 links, 7 joints
Joints:
- joint base: limit lower=-3.14 upper=3.14 effort=10 velocity=3.14 -> lower=-6.28318530717959 upper=6.28318530717959 effort=10 velocity=2.0943951023932
- joint elbow: limit lower=-3.14 upper=3.14 effort=10 velocity=3.14 -> lower=-2.87979326579064 upper=2.87979326579064 effort=10 velocity=3.14159265358979
- joint shoulder: limit lower=-3.14 upper=3.14 effort=10 velocity=3.14 -> lower=-6.28318530717959 upper=6.28318530717959 effort=10 velocity=2.0943951023932
- joint wrist1: limit lower=-3.14 upper=3.14 effort=10 velocity=3.14 -> lower=-6.28318530717959 upper=6.28318530717959 effort=10 velocity=3.14159265358979
- joint wrist2: limit lower=-3.14 upper=3.14 effort=10 velocity=3.14 -> lower=-6.28318530717959 upper=6.28318530717959 effort=10 velocity=3.14159265358979
- joint wrist3: limit lower=-3.14 upper=3.14 effort=10 velocity=3.14 -> lower=-6.28318530717959 upper=6.28318530717959 effort=10 velocity=3.14159265358979

File: rb_mujoco_ros2/rb_mujoco_description/urdf/rb16_900e_u.urdf (robot description, URDF)
Before this commit: robot rb16_900e_u, 8 links, 7 joints
Joints:
- joint base: limit lower=-3.14 upper=3.14 effort=10 velocity=3.14 -> lower=-6.28318530717959 upper=6.28318530717959 effort=10 velocity=2.0943951023932
- joint elbow: limit lower=-3.14 upper=3.14 effort=10 velocity=3.14 -> lower=-2.87979326579064 upper=2.87979326579064 effort=10 velocity=3.14159265358979
- joint shoulder: limit lower=-3.14 upper=3.14 effort=10 velocity=3.14 -> lower=-6.28318530717959 upper=6.28318530717959 effort=10 velocity=2.0943951023932
- joint wrist1: limit lower=-3.14 upper=3.14 effort=10 velocity=3.14 -> lower=-6.28318530717959 upper=6.28318530717959 effort=10 velocity=3.14159265358979
- joint wrist2: limit lower=-3.14 upper=3.14 effort=10 velocity=3.14 -> lower=-6.28318530717959 upper=6.28318530717959 effort=10 velocity=3.14159265358979
- joint wrist3: limit lower=-3.14 upper=3.14 effort=10 velocity=3.14 -> lower=-6.28318530717959 upper=6.28318530717959 effort=10 velocity=3.14159265358979

File: rb_mujoco_ros2/rb_mujoco_description/urdf/rb20_1800e_u.urdf (robot description, URDF)
Before this commit: robot rb20_1800e_u, 8 links, 7 joints
Joints:
- joint base: limit lower=-3.14 upper=3.14 effort=10 velocity=3.14 -> lower=-6.28318530717959 upper=6.28318530717959 effort=10 velocity=2.0943951023932
- joint elbow: limit lower=-3.14 upper=3.14 effort=10 velocity=3.14 -> lower=-2.87979326579064 upper=2.87979326579064 effort=10 velocity=3.14159265358979
- joint shoulder: limit lower=-3.14 upper=3.14 effort=10 velocity=3.14 -> lower=-6.28318530717959 upper=6.28318530717959 effort=10 velocity=2.0943951023932
- joint wrist1: limit lower=-3.14 upper=3.14 effort=10 velocity=3.14 -> lower=-6.28318530717959 upper=6.28318530717959 effort=10 velocity=3.14159265358979
- joint wrist2: limit lower=-3.14 upper=3.14 effort=10 velocity=3.14 -> lower=-6.28318530717959 upper=6.28318530717959 effort=10 velocity=3.14159265358979
- joint wrist3: limit lower=-3.14 upper=3.14 effort=10 velocity=3.14 -> lower=-6.28318530717959 upper=6.28318530717959 effort=10 velocity=3.14159265358979

File: rb_mujoco_ros2/rb_mujoco_description/urdf/rb20_1900es_u.urdf (robot description, URDF)
Before this commit: robot rb20_1900es_u, 8 links, 7 joints
Joints:
- joint base: limit lower=-3.14 upper=3.14 effort=10 velocity=3.14 -> lower=-6.28318530717959 upper=6.28318530717959 effort=10 velocity=2.0943951023932
- joint elbow: limit lower=-3.14 upper=3.14 effort=10 velocity=3.14 -> lower=-2.61799387799149 upper=2.61799387799149 effort=10 velocity=2.0943951023932
- joint shoulder: limit lower=-3.14 upper=3.14 effort=10 velocity=3.14 -> lower=-6.28318530717959 upper=6.28318530717959 effort=10 velocity=2.0943951023932
- joint wrist1: limit lower=-3.14 upper=3.14 effort=10 velocity=3.14 -> lower=-6.28318530717959 upper=6.28318530717959 effort=10 velocity=2.0943951023932
- joint wrist2: limit lower=-3.14 upper=3.14 effort=10 velocity=3.14 -> lower=-6.28318530717959 upper=6.28318530717959 effort=10 velocity=3.14159265358979
- joint wrist3: limit lower=-3.14 upper=3.14 effort=10 velocity=3.14 -> lower=-6.28318530717959 upper=6.28318530717959 effort=10 velocity=3.14159265358979

File: rb_mujoco_ros2/rb_mujoco_description/urdf/rb30_1400es_u.urdf (robot description, URDF)
Before this commit: robot rb30_1400es_u, 8 links, 7 joints
Joints:
- joint base: limit lower=-3.14 upper=3.14 effort=10 velocity=3.14 -> lower=-6.28318530717959 upper=6.28318530717959 effort=10 velocity=2.0943951023932
- joint elbow: limit lower=-3.14 upper=3.14 effort=10 velocity=3.14 -> lower=-2.61799387799149 upper=2.61799387799149 effort=10 velocity=2.0943951023932
- joint shoulder: limit lower=-3.14 upper=3.14 effort=10 velocity=3.14 -> lower=-6.28318530717959 upper=6.28318530717959 effort=10 velocity=2.0943951023932
- joint wrist1: limit lower=-3.14 upper=3.14 effort=10 velocity=3.14 -> lower=-6.28318530717959 upper=6.28318530717959 effort=10 velocity=2.0943951023932
- joint wrist2: limit lower=-3.14 upper=3.14 effort=10 velocity=3.14 -> lower=-6.28318530717959 upper=6.28318530717959 effort=10 velocity=3.14159265358979
- joint wrist3: limit lower=-3.14 upper=3.14 effort=10 velocity=3.14 -> lower=-6.28318530717959 upper=6.28318530717959 effort=10 velocity=3.14159265358979

File: rb_mujoco_ros2/rb_mujoco_description/urdf/rb3_1200e.urdf (robot description, URDF)
Before this commit: robot rb3_1200e, 8 links, 7 joints
Joints:
- joint base: limit lower=-3.14 upper=3.14 effort=10 velocity=3.14 -> lower=-6.28318530717959 upper=6.28318530717959 effort=10 velocity=3.14159265358979
- joint elbow: limit lower=-3.14 upper=3.14 effort=10 velocity=3.14 -> lower=-2.87979326579064 upper=2.87979326579064 effort=10 velocity=3.14159265358979
- joint shoulder: limit lower=-3.14 upper=3.14 effort=10 velocity=3.14 -> lower=-6.28318530717959 upper=6.28318530717959 effort=10 velocity=3.14159265358979
- joint wrist1: limit lower=-3.14 upper=3.14 effort=10 velocity=3.14 -> lower=-6.28318530717959 upper=6.28318530717959 effort=10 velocity=3.14159265358979
- joint wrist2: limit lower=-3.14 upper=3.14 effort=10 velocity=3.14 -> lower=-6.28318530717959 upper=6.28318530717959 effort=10 velocity=3.14159265358979
- joint wrist3: limit lower=-3.14 upper=3.14 effort=10 velocity=3.14 -> lower=-6.28318530717959 upper=6.28318530717959 effort=10 velocity=3.14159265358979

File: rb_mujoco_ros2/rb_mujoco_description/urdf/rb3_1200e_u.urdf (robot description, URDF)
Before this commit: robot rb3_1200e_u, 8 links, 7 joints
Joints:
- joint base: limit lower=-3.14 upper=3.14 effort=10 velocity=3.14 -> lower=-6.28318530717959 upper=6.28318530717959 effort=10 velocity=3.14159265358979
- joint elbow: limit lower=-3.14 upper=3.14 effort=10 velocity=3.14 -> lower=-2.87979326579064 upper=2.87979326579064 effort=10 velocity=3.14159265358979
- joint shoulder: limit lower=-3.14 upper=3.14 effort=10 velocity=3.14 -> lower=-6.28318530717959 upper=6.28318530717959 effort=10 velocity=3.14159265358979
- joint wrist1: limit lower=-3.14 upper=3.14 effort=10 velocity=3.14 -> lower=-6.28318530717959 upper=6.28318530717959 effort=10 velocity=3.14159265358979
- joint wrist2: limit lower=-3.14 upper=3.14 effort=10 velocity=3.14 -> lower=-6.28318530717959 upper=6.28318530717959 effort=10 velocity=3.14159265358979
- joint wrist3: limit lower=-3.14 upper=3.14 effort=10 velocity=3.14 -> lower=-6.28318530717959 upper=6.28318530717959 effort=10 velocity=3.14159265358979

File: rb_mujoco_ros2/rb_mujoco_description/urdf/rb3_730es_u.urdf (robot description, URDF)
Before this commit: robot rb3_730es_u, 8 links, 7 joints
Joints:
- joint base: limit lower=-3.14 upper=3.14 effort=10 velocity=3.14 -> lower=-6.28318530717959 upper=6.28318530717959 effort=10 velocity=3.14159265358979
- joint elbow: limit lower=-3.14 upper=3.14 effort=10 velocity=3.14 -> lower=-2.61799387799149 upper=2.61799387799149 effort=10 velocity=3.14159265358979
- joint shoulder: limit lower=-3.14 upper=3.14 effort=10 velocity=3.14 -> lower=-6.28318530717959 upper=6.28318530717959 effort=10 velocity=3.14159265358979
- joint wrist1: limit lower=-3.14 upper=3.14 effort=10 velocity=3.14 -> lower=-6.28318530717959 upper=6.28318530717959 effort=10 velocity=3.14159265358979
- joint wrist2: limit lower=-3.14 upper=3.14 effort=10 velocity=3.14 -> lower=-6.28318530717959 upper=6.28318530717959 effort=10 velocity=6.28318530717959
- joint wrist3: limit lower=-3.14 upper=3.14 effort=10 velocity=3.14 -> lower=-6.28318530717959 upper=6.28318530717959 effort=10 velocity=6.28318530717959

File: rb_mujoco_ros2/rb_mujoco_description/urdf/rb5_850e.urdf (robot description, URDF)
Before this commit: robot rb5_850e, 8 links, 7 joints
Joints:
- joint base: limit lower=-3.14 upper=3.14 effort=10 velocity=3.14 -> lower=-6.28318530717959 upper=6.28318530717959 effort=10 velocity=3.14159265358979
- joint elbow: limit lower=-3.14 upper=3.14 effort=10 velocity=3.14 -> lower=-2.87979326579064 upper=2.87979326579064 effort=10 velocity=3.14159265358979
- joint shoulder: limit lower=-3.14 upper=3.14 effort=10 velocity=3.14 -> lower=-6.28318530717959 upper=6.28318530717959 effort=10 velocity=3.14159265358979
- joint wrist1: limit lower=-3.14 upper=3.14 effort=10 velocity=3.14 -> lower=-6.28318530717959 upper=6.28318530717959 effort=10 velocity=3.14159265358979
- joint wrist2: limit lower=-3.14 upper=3.14 effort=10 velocity=3.14 -> lower=-6.28318530717959 upper=6.28318530717959 effort=10 velocity=3.14159265358979
- joint wrist3: limit lower=-3.14 upper=3.14 effort=10 velocity=3.14 -> lower=-6.28318530717959 upper=6.28318530717959 effort=10 velocity=3.14159265358979

File: rb_mujoco_ros2/rb_mujoco_description/urdf/rb5_850e_u.urdf (robot description, URDF)
Before this commit: robot rb5_850e_u, 8 links, 7 joints
Joints:
- joint base: limit lower=-3.14 upper=3.14 effort=10 velocity=3.14 -> lower=-6.28318530717959 upper=6.28318530717959 effort=10 velocity=3.14159265358979
- joint elbow: limit lower=-3.14 upper=3.14 effort=10 velocity=3.14 -> lower=-2.87979326579064 upper=2.87979326579064 effort=10 velocity=3.14159265358979
- joint shoulder: limit lower=-3.14 upper=3.14 effort=10 velocity=3.14 -> lower=-6.28318530717959 upper=6.28318530717959 effort=10 velocity=3.14159265358979
- joint wrist1: limit lower=-3.14 upper=3.14 effort=10 velocity=3.14 -> lower=-6.28318530717959 upper=6.28318530717959 effort=10 velocity=3.14159265358979
- joint wrist2: limit lower=-3.14 upper=3.14 effort=10 velocity=3.14 -> lower=-6.28318530717959 upper=6.28318530717959 effort=10 velocity=3.14159265358979
- joint wrist3: limit lower=-3.14 upper=3.14 effort=10 velocity=3.14 -> lower=-6.28318530717959 upper=6.28318530717959 effort=10 velocity=3.14159265358979

File: rb_mujoco_ros2/rb_mujoco_description/urdf/rb6_1700e_u.urdf (robot description, URDF)
Before this commit: robot rb6_1700e_u, 8 links, 7 joints
Joints:
- joint base: limit lower=-3.14 upper=3.14 effort=10 velocity=3.14 -> lower=-6.28318530717959 upper=6.28318530717959 effort=10 velocity=2.0943951023932
- joint elbow: limit lower=-3.14 upper=3.14 effort=10 velocity=3.14 -> lower=-2.79252680319093 upper=2.79252680319093 effort=10 velocity=3.14159265358979
- joint shoulder: limit lower=-3.14 upper=3.14 effort=10 velocity=3.14 -> lower=-6.28318530717959 upper=6.28318530717959 effort=10 velocity=2.0943951023932
- joint wrist1: limit lower=-3.14 upper=3.14 effort=10 velocity=3.14 -> lower=-6.28318530717959 upper=6.28318530717959 effort=10 velocity=3.14159265358979
- joint wrist2: limit lower=-3.14 upper=3.14 effort=10 velocity=3.14 -> lower=-6.28318530717959 upper=6.28318530717959 effort=10 velocity=3.14159265358979
- joint wrist3: limit lower=-3.14 upper=3.14 effort=10 velocity=3.14 -> lower=-6.28318530717959 upper=6.28318530717959 effort=10 velocity=3.14159265358979
