Commit message: feat(wuji): align flange mounts and expose Hand2 as beta2
Attach RB and RBY1 hands directly to flange frames, align Hand1 orientation in URDF and MJCF, and expose only wuji_hand/wuji_hand2 model choices. Extend mount and control checks across supported RBY1 versions. The existing rb20_1900es_u right-hand clearance failure remains documented.

File: rb_mujoco_ros2/rb_mujoco_description/urdf/rb_mujoco.urdf.xacro (robot description, xacro)
@@ -3,4 +3,11 @@
   <xacro:arg name="headless" default="false"/>
   <xacro:include filename="$(find rb_mujoco_description)/urdf/$(arg robot_model).urdf"/>
+  <!-- Joint zero: both thumbs +X, fingers +Z = TCP -Y; right dorsum +Y, left dorsum -Y. -->
+  <link name="flange"/>
+  <joint name="flange_joint" type="fixed">
+    <origin xyz="0 0 0" rpy="1.570796326794897 0 0"/>
+    <parent link="tcp"/>
+    <child link="flange"/>
+  </joint>
   <xacro:include filename="$(find rb_mujoco_description)/urdf/rb.ros2_control.xacro"/>
   <xacro:rb_ros2_control robot_model="$(arg robot_model)" headless="$(arg headless)"/>

File: rby1_mujoco_ros2/rby1_mujoco_description/urdf/rby1.ros2_control.xacro (robot description, xacro)
@@ -182,5 +182,5 @@
         <xacro:position_joint joint_name="left_finger5_joint4" initial_positions="${initial_positions}" />
       </xacro:if>
-      <xacro:if value="${(robot_model == 'a_wuji' or robot_model == 'm_wuji') and hand_model in ['wuji_hand2_beta1', 'wuji_hand2_beta2']}">
+      <xacro:if value="${(robot_model == 'a_wuji' or robot_model == 'm_wuji') and hand_model == 'wuji_hand2'}">
         <!-- Launch supplies the official Hand2 names and zero initial joint positions. -->
         <xacro:macro name="hand2_joints" params="names">

File: rby1_mujoco_ros2/rby1_mujoco_description/urdf/rby1.urdf.xacro (robot description, xacro)
@@ -8,5 +8,4 @@
   <xacro:arg name="mujoco_model_file" default="" />
   <xacro:arg name="headless" default="false" />
-  <xacro:arg name="hand_base_offset_z" default="0" />
   <xacro:property name="robot_model" value="$(arg robot_model)" />
   <xacro:property name="robot_version" value="$(arg robot_version)" />
@@ -20,10 +19,8 @@
     <xacro:include filename="$(find rby1_mujoco_description)/urdf/rby1m/model_${robot_version}.urdf" />
   </xacro:if>
+  <xacro:rby1_flange_frames />
   <xacro:if value="${robot_model == 'a_wuji' or robot_model == 'm_wuji'}">
     <xacro:rby1_wuji_hand_mounts robot_model="${robot_model}" robot_version="${robot_version}"
       hand_model="$(arg hand_model)" />
-  </xacro:if>
-  <xacro:if value="${robot_model != 'a_wuji' and robot_model != 'm_wuji'}">
-    <xacro:rby1_hand_base_frames hand_base_offset_z="$(arg hand_base_offset_z)" />
   </xacro:if>
   <!-- ros2_control -->

File: rby1_mujoco_ros2/rby1_mujoco_description/urdf/wuji_hand/left_with_docking.urdf.xacro (robot description, xacro)
@@ -1,5 +1,4 @@
 <?xml version="1.0"?>
 <robot xmlns:xacro="http://www.ros.org/wiki/xacro" name="rby1_wuji_hand_left">
-  <link name="left_hand_base" />
   <link name="left_hand_docking_link">
     <inertial>
@@ -29,12 +28,13 @@
   <xacro:include filename="$(find rby1_mujoco_description)/urdf/wuji_hand/left.urdf" />
   <joint name="left_wuji_mount_joint" type="fixed">
-    <parent link="left_hand_base" />
+    <parent link="left_flange" />
     <child link="left_hand_docking_link" />
-    <origin xyz="0.0 0.0 -0.02725" rpy="3.14159265359 0.0 2.35619449019" />
+    <!-- Adapter rotation aligns the native left thumb (-Y) with flange +X. -->
+    <origin xyz="0 0 ${0.02725 - hand_mount_offset_z}" rpy="0 0 3.141592653589793" />
   </joint>
   <joint name="left_hand_docking_joint" type="fixed">
     <parent link="left_hand_docking_link" />
     <child link="left_palm_link" />
-    <origin xyz="0.00065 0 0.022" rpy="0 0 -1.57079632679" />
+    <origin xyz="0.00065 0 0.022" rpy="0 0 -1.5707963267948966" />
   </joint>
 </robot>

File: rby1_mujoco_ros2/rby1_mujoco_description/urdf/wuji_hand/rby1_mount.urdf.xacro (robot description, xacro)
@@ -1,19 +1,22 @@
 <?xml version="1.0"?>
 <robot xmlns:xacro="http://www.ros.org/wiki/xacro">
-  <xacro:macro name="rby1_hand_base_frames" params="hand_base_offset_z:=0">
-    <link name="right_hand_base" />
-    <joint name="right_hand_base_joint" type="fixed">
+  <!-- Joint zero: thumb +X; left dorsum -Y, right dorsum +Y (outward); +Z = native -Z. -->
+  <xacro:macro name="rby1_flange_frames">
+    <link name="right_flange" />
+    <joint name="right_flange_joint" type="fixed">
       <parent link="ee_right" />
-      <child link="right_hand_base" />
-      <origin xyz="0 0 ${hand_base_offset_z}" rpy="0 0 0" />
+      <child link="right_flange" />
+      <origin xyz="0 0 0" rpy="3.141592653589793 0 0" />
     </joint>
-    <link name="left_hand_base" />
-    <joint name="left_hand_base_joint" type="fixed">
+    <link name="left_flange" />
+    <joint name="left_flange_joint" type="fixed">
       <parent link="ee_left" />
-      <child link="left_hand_base" />
-      <origin xyz="0 0 ${hand_base_offset_z}" rpy="0 0 0" />
+      <child link="left_flange" />
+      <origin xyz="0 0 0" rpy="3.141592653589793 0 0" />
     </joint>
   </xacro:macro>
   <xacro:macro name="rby1_wuji_hand_mounts" params="robot_model robot_version hand_model:=wuji_hand">
+    <xacro:property name="hand_mount_offset_z"
+      value="${0.066384 if robot_model == 'm_wuji' and robot_version == 'v1.3' else 0.0}" />
     <xacro:if value="${hand_model == 'wuji_hand'}">
       <xacro:include
@@ -22,34 +25,18 @@
         filename="$(find rby1_mujoco_description)/urdf/wuji_hand/left_with_docking.urdf.xacro" />
     </xacro:if>
-    <xacro:if value="${hand_model in ['wuji_hand2_beta1', 'wuji_hand2_beta2']}">
-      <xacro:include filename="$(find rby1_mujoco_description)/urdf/${hand_model}/right_with_mount-ros.urdf" />
-      <xacro:include filename="$(find rby1_mujoco_description)/urdf/${hand_model}/left_with_mount-ros.urdf" />
-      <link name="right_hand_base" />
-      <link name="left_hand_base" />
+    <xacro:if value="${hand_model == 'wuji_hand2'}">
+      <xacro:include filename="$(find rby1_mujoco_description)/urdf/wuji_hand2_beta2/right_with_mount-ros.urdf" />
+      <xacro:include filename="$(find rby1_mujoco_description)/urdf/wuji_hand2_beta2/left_with_mount-ros.urdf" />
       <joint name="right_wuji_mount_joint" type="fixed">
-        <parent link="right_hand_base" />
+        <parent link="right_flange" />
         <child link="r_mount" />
-        <origin xyz="0 0 0" rpy="0 0 0" />
+        <origin xyz="0 0 ${-hand_mount_offset_z}" rpy="3.141592653589793 0 0" />
       </joint>
       <joint name="left_wuji_mount_joint" type="fixed">
-        <parent link="left_hand_base" />
+        <parent link="left_flange" />
         <child link="l_mount" />
-        <origin xyz="0 0 0" rpy="0 0 0" />
+        <origin xyz="0 0 ${-hand_mount_offset_z}" rpy="3.141592653589793 0 0" />
       </joint>
     </xacro:if>
-    <joint name="right_hand_base_joint" type="fixed">
-      <parent link="ee_right" />
-      <child link="right_hand_base" />
-      <origin
-        xyz="${'0 0 0.066384' if robot_model == 'm_wuji' and robot_version == 'v1.3' else '0 0 0'}"
-        rpy="0 0 0" />
-    </joint>
-    <joint name="left_hand_base_joint" type="fixed">
-      <parent link="ee_left" />
-      <child link="left_hand_base" />
-      <origin
-        xyz="${'0 0 0.066384' if robot_model == 'm_wuji' and robot_version == 'v1.3' else '0 0 0'}"
-        rpy="0 0 0" />
-    </joint>
   </xacro:macro>
 </robot>

File: rby1_mujoco_ros2/rby1_mujoco_description/urdf/wuji_hand/right_with_docking.urdf.xacro (robot description, xacro)
@@ -1,5 +1,4 @@
 <?xml version="1.0"?>
 <robot xmlns:xacro="http://www.ros.org/wiki/xacro" name="rby1_wuji_hand_right">
-  <link name="right_hand_base" />
   <link name="right_hand_docking_link">
     <inertial>
@@ -29,12 +28,13 @@
   <xacro:include filename="$(find rby1_mujoco_description)/urdf/wuji_hand/right.urdf" />
   <joint name="right_wuji_mount_joint" type="fixed">
-    <parent link="right_hand_base" />
+    <parent link="right_flange" />
     <child link="right_hand_docking_link" />
-    <origin xyz="0.0 0.0 -0.02725" rpy="-3.14159265359 0.0 -2.35619449019" />
+    <!-- Adapter rotation aligns the native right thumb (+Y) with flange +X. -->
+    <origin xyz="0 0 ${0.02725 - hand_mount_offset_z}" rpy="0 0 3.141592653589793" />
   </joint>
   <joint name="right_hand_docking_joint" type="fixed">
     <parent link="right_hand_docking_link" />
     <child link="right_palm_link" />
-    <origin xyz="0.00065 0 0.022" rpy="0 0 1.57079632679" />
+    <origin xyz="0.00065 0 0.022" rpy="0 0 1.5707963267948966" />
   </joint>
 </robot>

File: rby1_mujoco_ros2/rby1_mujoco_description/urdf/wuji_hand2/hand.urdf.xacro (robot description, xacro)
@@ -2,14 +2,12 @@
 <robot xmlns:xacro="http://www.ros.org/wiki/xacro" name="rby1_wuji_hand2">
   <xacro:arg name="side" default="left" />
-  <xacro:arg name="hand_model" default="wuji_hand2_beta1" />
-  <xacro:property name="hand_model" value="$(arg hand_model)" />
   <xacro:property name="side" value="$(arg side)" />
-  <xacro:include filename="$(find rby1_mujoco_description)/urdf/${hand_model}/${side}_with_mount-ros.urdf" />
-  <link name="${side}_hand_base" />
+  <xacro:include filename="$(find rby1_mujoco_description)/urdf/wuji_hand2_beta2/${side}_with_mount-ros.urdf" />
+  <link name="${side}_flange" />
   <!-- Hand2 uses the official mount frame, without the Hand1 docking adapter. -->
   <joint name="${side}_wuji_mount_joint" type="fixed">
-    <parent link="${side}_hand_base" />
+    <parent link="${side}_flange" />
     <child link="${side[0]}_mount" />
-    <origin xyz="0 0 0" rpy="0 0 0" />
+    <origin xyz="0 0 0" rpy="3.141592653589793 0 0" />
   </joint>
 </robot>

Commit message: fix(rb): align flange and Wuji mounts with outward X

File: rb_mujoco_ros2/rb_mujoco_description/urdf/rb_mujoco.urdf.xacro (robot description, xacro)
@@ -3,8 +3,8 @@
   <xacro:arg name="headless" default="false"/>
   <xacro:include filename="$(find rb_mujoco_description)/urdf/$(arg robot_model).urdf"/>
-  <!-- Joint zero: both thumbs +X, fingers +Z = TCP -Y; right dorsum +Y, left dorsum -Y. -->
+  <!-- ROS-Industrial flange: +X outward; fixed right-handed Y/Z reference. -->
   <link name="flange"/>
   <joint name="flange_joint" type="fixed">
-    <origin xyz="0 0 0" rpy="1.570796326794897 0 0"/>
+    <origin xyz="0 0 0" rpy="0 0 -1.570796326794897"/>
     <parent link="tcp"/>
     <child link="flange"/>
