Commit message: fix(rby1): align flange axes while preserving hand poses

File: rby1_mujoco_ros2/rby1_mujoco_description/urdf/wuji_hand/left_with_docking.urdf.xacro (robot description, xacro)
@@ -30,6 +30,6 @@
     <parent link="left_flange" />
     <child link="left_hand_docking_link" />
-    <!-- Adapter rotation aligns the native left thumb (-Y) with flange +X. -->
-    <origin xyz="0 0 ${0.02725 - hand_mount_offset_z}" rpy="0 0 3.141592653589793" />
+    <!-- Fingers follow flange +X; thumb follows flange +Z. -->
+    <origin xyz="${0.02725 - hand_mount_offset_z} 0 0" rpy="0 1.570796326794897 0" />
   </joint>
   <joint name="left_hand_docking_joint" type="fixed">

File: rby1_mujoco_ros2/rby1_mujoco_description/urdf/wuji_hand/rby1_mount.urdf.xacro (robot description, xacro)
@@ -1,5 +1,5 @@
 <?xml version="1.0"?>
 <robot xmlns:xacro="http://www.ros.org/wiki/xacro">
-  <!-- Joint zero: thumb +X; left dorsum -Y, right dorsum +Y (outward); +Z = native -Z. -->
+  <!-- ROS-Industrial flange: +X = native -Z, +Y = native +Y, +Z = native +X. -->
   <xacro:macro name="rby1_flange_frames">
     <link name="right_flange" />
@@ -7,5 +7,5 @@
       <parent link="ee_right" />
       <child link="right_flange" />
-      <origin xyz="0 0 0" rpy="3.141592653589793 0 0" />
+      <origin xyz="0 0 0" rpy="0 1.570796326794897 0" />
     </joint>
     <link name="left_flange" />
@@ -13,5 +13,5 @@
       <parent link="ee_left" />
       <child link="left_flange" />
-      <origin xyz="0 0 0" rpy="3.141592653589793 0 0" />
+      <origin xyz="0 0 0" rpy="0 1.570796326794897 0" />
     </joint>
   </xacro:macro>
@@ -31,10 +31,10 @@
         <parent link="right_flange" />
         <child link="r_mount" />
-        <origin xyz="0 0 ${-hand_mount_offset_z}" rpy="3.141592653589793 0 0" />
+        <origin xyz="${-hand_mount_offset_z} 0 0" rpy="0 -1.570796326794897 0" />
       </joint>
       <joint name="left_wuji_mount_joint" type="fixed">
         <parent link="left_flange" />
         <child link="l_mount" />
-        <origin xyz="0 0 ${-hand_mount_offset_z}" rpy="3.141592653589793 0 0" />
+        <origin xyz="${-hand_mount_offset_z} 0 0" rpy="0 -1.570796326794897 0" />
       </joint>
     </xacro:if>

File: rby1_mujoco_ros2/rby1_mujoco_description/urdf/wuji_hand/right_with_docking.urdf.xacro (robot description, xacro)
@@ -30,6 +30,6 @@
     <parent link="right_flange" />
     <child link="right_hand_docking_link" />
-    <!-- Adapter rotation aligns the native right thumb (+Y) with flange +X. -->
-    <origin xyz="0 0 ${0.02725 - hand_mount_offset_z}" rpy="0 0 3.141592653589793" />
+    <!-- Fingers follow flange +X; thumb follows flange +Z. -->
+    <origin xyz="${0.02725 - hand_mount_offset_z} 0 0" rpy="0 1.570796326794897 0" />
   </joint>
   <joint name="right_hand_docking_joint" type="fixed">

File: rby1_mujoco_ros2/rby1_mujoco_description/urdf/wuji_hand2/hand.urdf.xacro (robot description, xacro)
@@ -9,5 +9,5 @@
     <parent link="${side}_flange" />
     <child link="${side[0]}_mount" />
-    <origin xyz="0 0 0" rpy="3.141592653589793 0 0" />
+    <origin xyz="0 0 0" rpy="0 -1.570796326794897 0" />
   </joint>
 </robot>
